File: prototype/ErgoSNM_Keyboard_Left_Prototype_1/ErgoSNM_Keyboard_Left_Prototype_1.kicad_pcb (KiCad board)
At the start: 2 copper layers, 67 parts, among them J1 Conn_01x02, J2 Conn_01x02, J3 Conn_01x02, J4 Conn_01x06, J5 Conn_01x05, M1 nRF51822_Core_board, M2 Pro_Micro, M3 Adafruit_Bluefruit_LE_SPI_Fri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, SW1 SW_Push, SW2 SW_2P3T, U1 TP4057

Commit message: Update PCB
Parts:
- added REF**: MountingHole_2.2mm_M2_DIN965, MountingHole:MountingHole_2.2mm_M2_DIN965, F.Cu at (89.0, 143.0)
- added REF**: MountingHole_2.2mm_M2_DIN965, MountingHole:MountingHole_2.2mm_M2_DIN965, F.Cu at (89.0, 60.0)
- added REF**: MountingHole_2.2mm_M2_DIN965, MountingHole:MountingHole_2.2mm_M2_DIN965, F.Cu at (224.0, 60.0)
- added REF**: MountingHole_2.2mm_M2_DIN965, MountingHole:MountingHole_2.2mm_M2_DIN965, F.Cu at (224.0, 143.0)
- C1, C2: footprint Capacitor_SMD:C_0201_0603Metric_Pad0.64x0.40mm_HandSolder -> Capacitor_SMD:C_0603_1608Metric_Pad1.08x0.95mm_HandSolder; moved to B.Cu
- D1, D10, D11, D12, D13, D14, D15, D16, D17, D18, D19, D2, D20, D21, D22, D23, D24, D3, D4, D5, D6, D7, D8, D9, J1, J3, JP1, M1, M3, SW1, SW2, U1: moved to B.Cu
- D25: footprint Diode_THT:D_DO-41_SOD81_P10.16mm_Horizontal -> Diode_SMD:D_1206_3216Metric_Pad1.42x1.75mm_HandSolder; moved to B.Cu
- J2: footprint Connector_PinHeader_2.54mm:PinHeader_1x02_P2.54mm_Horizontal -> Connector_PinHeader_2.54mm:PinHeader_1x02_P2.54mm_Vertical
- R1, R2: footprint Resistor_SMD:R_0201_0603Metric_Pad0.64x0.40mm_HandSolder -> Capacitor_SMD:C_0603_1608Metric_Pad1.08x0.95mm_HandSolder; moved to B.Cu
- moved J3 134.4 mm to (192.8, 66.0)
- moved C1 130.9 mm to (201.7, 72.0)
- moved D25 128.6 mm to (187.5, 66.0), turned to -90 degrees
- moved C2 122.2 mm to (200.5, 64.0), turned to 90 degrees
- moved U1 116.7 mm to (201.7, 68.2), turned to 90 degrees
- moved R2 113.6 mm to (223.2, 109.0), turned to 180 degrees
- moved R1 112.9 mm to (203.0, 64.0), turned to 90 degrees
- moved M2 111.7 mm to (215.4, 77.9), turned to -90 degrees
- moved M1 105.1 mm to (213.0, 120.0), turned to 90 degrees
- moved J2 104.0 mm to (201.5, 77.5), turned to 180 degrees
- moved KEY12 100.1 mm to (190.5, 95.2)
- moved KEY6 99.9 mm to (190.5, 76.2)
- moved D23 92.2 mm to (179.1, 142.2), turned to 90 degrees
- moved KEY22 88.1 mm to (152.4, 133.3)
- moved D6 87.6 mm to (198.1, 85.1), turned to 90 degrees
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Connections:
- SW2 pad 1: /RAW_Pro_Micro -> Net-(D25-Pad1)
- SW2 pad 2: Net-(D25-Pad1) -> unconnected-(SW2-Pad2)
- SW2 pad 3: unconnected-(SW2-Pad3) -> /RAW_Pro_Micro
- SW2 pad 5: +3V3 -> /2.4GHz_Enable
- SW2 pad 6: /2.4GHz_Enable -> Net-(JP1-Pad1)
- SW2 pad 7: Net-(JP1-Pad1) -> +3V3
- SWD1 pad 2: Net-(M1-Pad31) -> Net-(M1-Pad32)
- SWD1 pad 3: Net-(M1-Pad32) -> Net-(M1-Pad31)
Routing:
- net /Col_0: track 0.00 -> 252.2 mm
- net /Col_1: track 0.00 -> 218.3 mm
- net /Col_2: track 0.00 -> 195.6 mm
- net +3V3: track 0.00 -> 190.0 mm
- net /Col_3: track 0.00 -> 178.3 mm
- net /Row_1: track 0.00 -> 152.1 mm
- net /Row_0: track 0.00 -> 151.4 mm
- net /Row_2: track 0.00 -> 147.4 mm
- net /Col_4: track 0.00 -> 146.1 mm
- net /Row_3: track 0.00 -> 133.6 mm
- net /Col_5: track 0.00 -> 126.3 mm
- net /RST_Pro_Micro: track 0.00 -> 110.2 mm
- net /2.4GHz_Enable: track 0.00 -> 78.7 mm
- net /Tx_nRF5: track 0.00 -> 65.9 mm
- net /Rx_nRF5: track 0.00 -> 64.9 mm
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- added copper zone on B.Cu, net GND
- added copper zone on F.Cu, net GND
Other:
- board outline added: 140 x 88 mm
- board text added: "2.4G-USB-BT"
- board text added: "3.3V SCK MOSI MISO CS GND"
- board text added: "3.3V SWCLK SWDIO GND"
- board text added: "BT-USB-2.4G"
- board text added: "ErgoSNM Keyboard (Left) Prototype Rev.1"
- board text added: "P0.12 P0.13 P0.14 P0.30 P0.28"
- board text added: "RESET"
- board text added: "SCK MISO MOSI CS IRQ DFU RST GND VIN"
