File: prototype/ErgoSNM_Keyboard_Left_Prototype_1/ErgoSNM_Keyboard_Left_Prototype_1.kicad_sch (KiCad schematic)
At the start: 0 parts

Commit message: Update Sch file
Parts:
- added C1: 10uF, Capacitor_SMD:C_0201_0603Metric_Pad0.64x0.40mm_HandSolder, symbol Device:C_Small
- added C2: 1uF, Capacitor_SMD:C_0201_0603Metric_Pad0.64x0.40mm_HandSolder, symbol Device:C_Small
- added D1, D10, D11, D12, D13, D14, D15, D16, D17, D18, D19, D2, D20, D21, D22, D23, D24, D3, D4, D5, D6, D7, D8, D9: 1N4148, Diode_SMD:D_0603_1608Metric_Pad1.05x0.95mm_HandSolder, symbol Diode:1N4148
- added D25: 1N5819, Diode_THT:D_DO-41_SOD81_P10.16mm_Horizontal, symbol Diode:1N5819
- added J1, J2: Conn_01x02, Connector_PinHeader_2.54mm:PinHeader_1x02_P2.54mm_Horizontal, symbol Connector_Generic:Conn_01x02
- added J3: Conn_01x02, Connector_JST:JST_EH_B2B-EH-A_1x02_P2.50mm_Vertical, symbol Connector_Generic:Conn_01x02
- added J4: Conn_01x06, Connector_PinHeader_2.54mm:PinHeader_1x06_P2.54mm_Vertical, symbol Connector_Generic:Conn_01x06
- added J5: Conn_01x05, Connector_PinHeader_2.54mm:PinHeader_1x05_P2.54mm_Vertical, symbol Connector_Generic:Conn_01x05
- added JP1: Jumper_2_Bridged, Jumper:SolderJumper-2_P1.3mm_Open_TrianglePad1.0x1.5mm, symbol Jumper:Jumper_2_Bridged
- added KEY1: 00, key-switches:MX_Switch_Gateron_socket_A, symbol Switch:SW_Push_45deg
- added KEY10: 13, key-switches:MX_Switch_Gateron_socket_A, symbol Switch:SW_Push_45deg
- added KEY11: 14, key-switches:MX_Switch_Gateron_socket_A, symbol Switch:SW_Push_45deg
- added KEY12: 15, key-switches:MX_Switch_Gateron_socket_A, symbol Switch:SW_Push_45deg
- added KEY13: 20, key-switches:MX_Switch_Gateron_socket_A, symbol Switch:SW_Push_45deg
- added KEY14: 21, key-switches:MX_Switch_Gateron_socket_A, symbol Switch:SW_Push_45deg
- added KEY15: 22, key-switches:MX_Switch_Gateron_socket_A, symbol Switch:SW_Push_45deg
- added KEY16: 23, key-switches:MX_Switch_Gateron_socket_A, symbol Switch:SW_Push_45deg
- added KEY17: 24, key-switches:MX_Switch_Gateron_socket_A, symbol Switch:SW_Push_45deg
- added KEY18: 25, key-switches:MX_Switch_Gateron_socket_A, symbol Switch:SW_Push_45deg
- added KEY19: 30, key-switches:MX_Switch_Gateron_socket_A, symbol Switch:SW_Push_45deg
- added KEY2: 01, key-switches:MX_Switch_Gateron_socket_A, symbol Switch:SW_Push_45deg
- added KEY20: 31, key-switches:MX_Switch_Gateron_socket_A, symbol Switch:SW_Push_45deg
- added KEY21: 32, key-switches:MX_Switch_Gateron_socket_A, symbol Switch:SW_Push_45deg
- added KEY22: 33, key-switches:MX_Switch_Gateron_socket_A, symbol Switch:SW_Push_45deg
- added KEY23: 34, key-switches:MX_Switch_Gateron_socket_A, symbol Switch:SW_Push_45deg
- added KEY24: 35, key-switches:MX_Switch_Gateron_socket_A, symbol Switch:SW_Push_45deg
- added KEY3: 02, key-switches:MX_Switch_Gateron_socket_A, symbol Switch:SW_Push_45deg
- added KEY4: 03, key-switches:MX_Switch_Gateron_socket_A, symbol Switch:SW_Push_45deg
- added KEY5: 04, key-switches:MX_Switch_Gateron_socket_A, symbol Switch:SW_Push_45deg
- added KEY6: 05, key-switches:MX_Switch_Gateron_socket_A, symbol Switch:SW_Push_45deg
- added KEY7: 10, key-switches:MX_Switch_Gateron_socket_A, symbol Switch:SW_Push_45deg
- added KEY8: 11, key-switches:MX_Switch_Gateron_socket_A, symbol Switch:SW_Push_45deg
- added KEY9: 12, key-switches:MX_Switch_Gateron_socket_A, symbol Switch:SW_Push_45deg
- added M1: nRF51822_Core_board, ErgoSNM_Keybaord:Core51822, symbol ErgoSNM_Keybaord_Library:nRF51822_Core_board
- added M2: Pro_Micro, ErgoSNM_Keybaord:Pro_Micro, symbol ErgoSNM_Keybaord_Library:Pro_Micro
- added M3: Adafruit_Bluefruit_LE_SPI_Friend, Connector_PinHeader_2.54mm:PinHeader_1x09_P2.54mm_Vertical, symbol ErgoSNM_Keybaord_Library:Adafruit_Bluefruit_LE_SPI_Friend
- added R1: 4.7k, Resistor_SMD:R_0201_0603Metric_Pad0.64x0.40mm_HandSolder, symbol Device:R
- added R2: 10k, Resistor_SMD:R_0201_0603Metric_Pad0.64x0.40mm_HandSolder, symbol Device:R
- added SW1: SW_Push, Button_Switch_SMD:SW_Push_1P1T_NO_CK_KSC6xxJ, symbol Switch:SW_Push
- added SW2: SW_2P3T, ErgoSNM_Keybaord:MSK-23D20-T, symbol ErgoSNM_Keybaord_Library:SW_2P3T
- added SWD1: Conn_01x04, Connector_PinHeader_2.54mm:PinHeader_1x04_P2.54mm_Horizontal, symbol Connector_Generic:Conn_01x04
- added TRRS1: PJ-393_TRRS_8P, ErgoSNM_Keybaord:PJ-393, symbol ErgoSNM_Keybaord_Library:PJ-393_TRRS_8P
- added U1: TP4057, Package_TO_SOT_SMD:SOT-23-6_Handsoldering, symbol ErgoSNM_Keybaord_Library:TP4057
Connections:
- new net: D1.2 (A), KEY1.2
- new net: M1.31 (SWDIO/RESET), SWD1.2 (Pin_2)
- new net: M1.32 (SWCLK), SWD1.3 (Pin_3)
- new net: D17.2 (A), KEY17.2
- new net: D14.2 (A), KEY14.2
- new net: D3.2 (A), KEY3.2
- new net: D22.2 (A), KEY22.2
- new net: D23.2 (A), KEY23.2
- new net: D8.2 (A), KEY8.2
- new net: D13.2 (A), KEY13.2
- new net: D16.2 (A), KEY16.2
- new net: D5.2 (A), KEY5.2
- new net: D10.2 (A), KEY10.2
- new net: JP1.1 (A), SW2.7
- new net: D7.2 (A), KEY7.2
- new net: D11.2 (A), KEY11.2
- new net: D24.2 (A), KEY24.2
- new net: J2.1 (Pin_1), U1.1 (CHRG)
- new net: J2.2 (Pin_2), U1.5 (STDBY)
- new net: D12.2 (A), KEY12.2
- new net: D15.2 (A), KEY15.2
- new net: D19.2 (A), KEY19.2
- new net: J5.1 (Pin_1), M1.12 (P0.12)
- new net: J5.2 (Pin_2), M1.13 (P0.13)
- new net: J5.3 (Pin_3), M1.14 (P0.14)
- new net: J5.5 (Pin_5), M1.28 (P0.28)
- new net: J5.4 (Pin_4), M1.30 (P0.30)
- new net: R1.1, U1.6 (PROG)
- new net: D25.1 (K), SW2.2, SW2.4
- new net: D9.2 (A), KEY9.2
- new net: D4.2 (A), KEY4.2
- new net: D2.2 (A), KEY2.2
- new net: D18.2 (A), KEY18.2
- new net: D20.2 (A), KEY20.2
- new net: D21.2 (A), KEY21.2
- new net: D6.2 (A), KEY6.2
- new net +3V3: J4.1 (Pin_1), M1.33 (Vcc), M2.Vcc, SW2.5, SWD1.1 (Pin_1), TRRS1.8 (Sa)
- new net 2.4GHz_Enable: M1.6 (P0.06), R2.1, SW2.6
- new net CS_Bluefruit: M2.8 (D8A8/PB4), M3.4 (CS)
- new net CS_nRF5: J4.5 (Pin_5), M1.4 (P0.04)
- new net Col_0: KEY1.1, KEY13.1, KEY19.1, KEY7.1, M1.20 (P0.20)
- new net Col_1: KEY14.1, KEY2.1, KEY20.1, KEY8.1, M1.21 (P0.21)
- new net Col_2: KEY15.1, KEY21.1, KEY3.1, KEY9.1, M1.22 (P0.22)
- new net Col_3: KEY10.1, KEY16.1, KEY22.1, KEY4.1, M1.23 (P0.23)
- new net Col_4: KEY11.1, KEY17.1, KEY23.1, KEY5.1, M1.24 (P0.24)
- new net Col_5: KEY12.1, KEY18.1, KEY24.1, KEY6.1, M1.25 (P0.25)
- new net GND: C1.2, C2.2, J1.2 (Pin_2), J3.2 (Pin_2), J4.6 (Pin_6), M1.34 (GND), M2.GND0 (GND), M2.GND1 (GND), M2.GND2 (GND), M3.8 (GND), R1.2, R2.2, SW1.1, SWD1.4 (Pin_4), TRRS1.1 (Ta), U1.2 (GND)
- new net IRQ_Bluefruit: M2.7 (D7/PE6), M3.5 (IRQ)
- new net MISO_Bluefruit: M2.14 (D14/PB3), M3.2 (MISO)
- new net MISO_nRF5: J4.4 (Pin_4), M1.3 (P0.03), TRRS1.3 (R2a)
- new net MOSI_Bluefruit: M2.16 (D16/PB2), M3.3 (MOSI)
- new net MOSI_nRF5: J4.3 (Pin_3), M1.2 (P0.02)
- new net RAW_Pro_Micro: C2.1, M2.RAW, SW2.1, U1.4 (Vcc)
- new net RST_Bluefruit: M2.4 (D4A6/PD4), M3.7 (RST/SWDIO)
- new net RST_Pro_Micro: J1.1 (Pin_1), M2.RST (Reset), SW1.2
- new net Row_0: D1.1 (K), D2.1 (K), D3.1 (K), D4.1 (K), D5.1 (K), D6.1 (K), M1.15 (P0.15)
- new net Row_1: D10.1 (K), D11.1 (K), D12.1 (K), D7.1 (K), D8.1 (K), D9.1 (K), M1.16 (P0.16)
- new net Row_2: D13.1 (K), D14.1 (K), D15.1 (K), D16.1 (K), D17.1 (K), D18.1 (K), M1.17 (P0.17)
- new net Row_3: D19.1 (K), D20.1 (K), D21.1 (K), D22.1 (K), D23.1 (K), D24.1 (K), M1.18 (P0.18)
- new net Rx_nRF5: M1.11 (P0.11), M2.0 (D0/PD2)
- new net SCK_Bluefruit: M2.15 (D15/PB1), M3.1 (SCK)
- new net SCK_nRF5: J4.2 (Pin_2), M1.1 (P0.01), TRRS1.2 (R1a)
- new net Tx_nRF5: M1.9 (P0.09), M2.1 (D1/PD3)
- new net Vcc_BATT: C1.1, D25.2 (A), J3.1 (Pin_1), U1.3 (BAT)
- new net Vcc_Bluefruit: JP1.2 (B), M3.9 (VIN), SW2.8
- no-connect marks 0 -> 8
Other:
- note added: "2/6: 2.4GHz 3/7: USB (Battery off) 4/8: Bluetooth"

Commit message: Update PCB
Parts:
- D25: footprint Diode_THT:D_DO-41_SOD81_P10.16mm_Horizontal -> Diode_SMD:D_1206_3216Metric_Pad1.42x1.75mm_HandSolder
- J2: footprint Connector_PinHeader_2.54mm:PinHeader_1x02_P2.54mm_Horizontal -> Connector_PinHeader_2.54mm:PinHeader_1x02_P2.54mm_Vertical
Connections:
- net +3V3: now also SW2.7; no longer SW2.5
- net 2.4GHz_Enable: now also SW2.5; no longer SW2.6
- net RAW_Pro_Micro: now also SW2.3; no longer SW2.1
- net at SWD1.2 (Pin_2): now also M1.32 (SWCLK); no longer M1.31 (SWDIO/RESET)
- net at SWD1.3 (Pin_3): now also M1.31 (SWDIO/RESET); no longer M1.32 (SWCLK)
- net at JP1.1 (A): now also SW2.6; no longer SW2.7
- net at D25.1 (K), SW2.4: now also SW2.1; no longer SW2.2
Other:
- note added: "1/5: 2.4GHz 2/6: USB (Battery off) 4/8: Bluetooth"
- note removed: "2/6: 2.4GHz 3/7: USB (Battery off) 4/8: Bluetooth"
Changed lines of the file:
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@@
+    (stroke (width 0) (type default) (color 0 0 0 0))
+  )
+  (wire (pts (xy 66.04 27.94) (xy 74.93 27.94))
     (stroke (width 0) (type default) (color 0 0 0 0))
   )
@@
     (stroke (width 0) (type default) (color 0 0 0 0))
   )
+  (wire (pts (xy 74.93 27.94) (xy 85.09 30.48))
+    (stroke (width 0) (type default) (color 0 0 0 0))
+  )
   (bus (pts (xy 80.01 137.16) (xy 80.01 177.8))
     (stroke (width 0) (type default) (color 0 0 0 0))
@@
     (stroke (width 0) (type default) (color 0 0 0 0))
   )
-  (wire (pts (xy 66.04 30.48) (xy 85.09 30.48))
-    (stroke (width 0) (type default) (color 0 0 0 0))
-  )
   (wire (pts (xy 21.59 35.56) (xy 36.83 35.56))
     (stroke (width 0) (type default) (color 0 0 0 0))
@@
     (stroke (width 0) (type default) (color 0 0 0 0))
   )
+  (wire (pts (xy 74.93 30.48) (xy 85.09 27.94))
+    (stroke (width 0) (type default) (color 0 0 0 0))
+  )
   (wire (pts (xy 265.43 30.48) (xy 265.43 48.26))
     (stroke (width 0) (type default) (color 0 0 0 0))
@@
     (stroke (width 0) (type default) (color 0 0 0 0))
   )
-  (wire (pts (xy 66.04 27.94) (xy 85.09 27.94))
-    (stroke (width 0) (type default) (color 0 0 0 0))
-  )
   (wire (pts (xy 21.59 60.96) (xy 36.83 60.96))
     (stroke (width 0) (type default) (color 0 0 0 0))
@@
     (stroke (width 0) (type default) (color 0 0 0 0))
   )
+  (wire (pts (xy 66.04 30.48) (xy 74.93 30.48))
+    (stroke (width 0) (type default) (color 0 0 0 0))
+  )
   (wire (pts (xy 21.59 58.42) (xy 36.83 58.42))
     (stroke (width 0) (type default) (color 0 0 0 0))
@@
     (stroke (width 0) (type default) (color 0 0 0 0))
   )
-  (text "2/6: 2.4GHz\n3/7: USB (Battery off)\n4/8: Bluetooth" (at 234.95 119.38 0)
+  (text "1/5: 2.4GHz\n2/6: USB (Battery off)\n4/8: Bluetooth" (at 234.95 119.38 0)
     (effects (font (size 1.27 1.27)) (justify left bottom))
   )
@@
     (property "Reference" "J2" (id 0) (at 163.83 123.19 0))
     (property "Value" "Conn_01x02" (id 1) (at 163.83 125.73 0))
-    (property "Footprint" "Connector_PinHeader_2.54mm:PinHeader_1x02_P2.54mm_Horizontal" (id 2) (at 163.83 129.54 0)
+    (property "Footprint" "Connector_PinHeader_2.54mm:PinHeader_1x02_P2.54mm_Vertical" (id 2) (at 163.83 129.54 0)
       (effects (font (size 1.27 1.27)) hide)
     )
@@
     (property "Reference" "D25" (id 0) (at 261.3025 124.46 0))
     (property "Value" "1N5819" (id 1) (at 261.3025 127 0))
-    (property "Footprint" "Diode_THT:D_DO-41_SOD81_P10.16mm_Horizontal" (id 2) (at 261.62 135.255 0)
+    (property "Footprint" "Diode_SMD:D_1206_3216Metric_Pad1.42x1.75mm_HandSolder" (id 2) (at 261.62 135.255 0)
       (effects (font (size 1.27 1.27)) hide)
     )
@@
       (effects (font (size 1.27 1.27)) hide)
     )
-    (pin "1")
-    (pin "2")
     (pin "3")
+    (pin "1")
+    (pin "2")
     (pin "4")
+    (pin "7")
     (pin "5")
     (pin "6")
-    (pin "7")
     (pin "8")
   )
@@
     )
     (path "/9e72a9c2-0df9-4b1f-b010-9c2cf2337a45"
-      (reference "D25") (unit 1) (value "1N5819") (footprint "Diode_THT:D_DO-41_SOD81_P10.16mm_Horizontal")
+      (reference "D25") (unit 1) (value "1N5819") (footprint "Diode_SMD:D_1206_3216Metric_Pad1.42x1.75mm_HandSolder")
     )
     (path "/0da70b93-f6fd-43b0-ad16-028b2909078c"
@@
     )
     (path "/66d4feec-1111-44d2-86dd-039c501ff49c"
-      (reference "J2") (unit 1) (value "Conn_01x02") (footprint "Connector_PinHeader_2.54mm:PinHeader_1x02_P2.54mm_Horizontal")
+      (reference "J2") (unit 1) (value "Conn_01x02") (footprint "Connector_PinHeader_2.54mm:PinHeader_1x02_P2.54mm_Vertical")
     )
     (path "/53c4fade-383c-48e4-915b-383f08dbc595"
