File: ErgoSNM_Keyboard/ErgoSNM_keyboard.kicad_pcb (KiCad board)
At the start: 2 copper layers, 173.1 x 137.3 mm, 114 parts, among them J1 Conn_01x13, J2 Conn_01x13, J3 Conn_01x06, J4 Conn_01x04, J5 Conn_01x07, J6 Conn_01x03, J7 Conn_01x07, SW1 RESET, SW2 SW_2P2T

Commit message: Update footprint
Parts:
- KEY1, KEY10, KEY11, KEY12, KEY13, KEY14, KEY15, KEY16, KEY17, KEY18, KEY19, KEY2, KEY20, KEY21, KEY22, KEY23, KEY24, KEY25, KEY26, KEY27, KEY28, KEY29, KEY3, KEY30, KEY31, KEY32, KEY33, KEY34, KEY35, KEY4, KEY5, KEY6, KEY7, KEY8, KEY9: footprint key-switches:MX_switch_Gateron_hotswap_double_sided_A -> key-switches:MX_switch_THT_hotswap_double_sided_A
Connections:
- net SCL renamed ENC_B
