File: ErgoSNM_Keyboard/ErgoSNM_keyboard.kicad_sch (KiCad schematic)
At the start: 96 parts, among them J1 Conn_01x13, J2 Conn_01x13, J3 Conn_01x03, J4 Conn_01x04, SW1 RESET, SW2 SW_2P2T

Commit message: Update PCB
Parts:
- added J3: Conn_01x06, Connector_PinHeader_2.54mm:PinHeader_1x06_P2.54mm_Vertical, symbol Connector_Generic:Conn_01x06
- added J5, J7: Conn_01x07, Connector_PinHeader_2.54mm:PinHeader_1x07_P2.54mm_Vertical, symbol Connector_Generic:Conn_01x07
- J6: renamed from J3; footprint Connector_JST:JST_PH_B2B-PH-K_1x02_P2.00mm_Vertical -> Connector_JST:JST_PH_B3B-PH-K_1x03_P2.00mm_Vertical
- renumbered D11 to D10, D12 to D11, D13 to D12, D14 to D13, D15 to D14, D16 to D15, D17 to D16, D18 to D17, D19 to D18, D20 to D19, D21 to D20, D22 to D21, D23 to D22, D24 to D23, D25 to D24, D26 to D25, D27 to D26, D28 to D27, D29 to D28, D30 to D29, D31 to D30, D32 to D31, D33 to D32, D34 to D33, D35 to D34, D36 to D35, D9 to D8, D10 to D9, D8 to LD1, TP11 to TP10, TP12 to TP11, TP13 to TP12, TP14 to TP13, TP6 to TP14, TP5 to TP4, TP7 to TP5, TP4 to TP6, TP8 to TP7, TP9 to TP8, TP10 to TP9
Connections:
- net COL_5: now also J5.7 (Pin_7), J7.7 (Pin_7)
- net COL_6: now also J4.3 (Pin_3), J5.1 (Pin_1), J7.1 (Pin_1)
- net CS: now also J3.6 (Pin_6); no longer J4.1 (Pin_1)
- net GND: now also J4.2 (Pin_2), J3.2 (Pin_2)
- net MISO: now also J3.4 (Pin_4); no longer J4.3 (Pin_3)
- net MOSI: now also J3.5 (Pin_5); no longer J4.2 (Pin_2)
- net ROW_0: now also J5.2 (Pin_2), J7.2 (Pin_2)
- net ROW_1: now also J5.3 (Pin_3), J7.3 (Pin_3)
- net ROW_2: now also J5.4 (Pin_4), J7.4 (Pin_4)
- net ROW_3: now also J5.5 (Pin_5), J7.5 (Pin_5)
- net ROW_4: now also J5.6 (Pin_6), J7.6 (Pin_6)
- net SCLK: now also J3.3 (Pin_3); no longer J4.4 (Pin_4)
- net SDA: now also R4.1, TP14.1, TRRS1.2 (R1a); no longer R3.2, TP6.1, TRRS1.3 (R2a)
- net VCC: now also J4.1 (Pin_1), J3.1 (Pin_1)
- removed net SCL: J1.7 (Pin_7), R4.1, TP14.1, TRRS1.2 (R1a)
- new net ENC_B: J1.7 (Pin_7), J4.4 (Pin_4), R3.2, TP6.1, TRRS1.3 (R2a)
Other:
- moved on the sheet: J1, J2, J6, LD1, R1, R2, R3, R4, SW1, SW2, TP14, TP6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

Commit message: Update footprint
Parts:
- KEY1, KEY10, KEY11, KEY12, KEY13, KEY14, KEY15, KEY16, KEY17, KEY18, KEY19, KEY2, KEY20, KEY21, KEY22, KEY23, KEY24, KEY25, KEY26, KEY27, KEY28, KEY29, KEY3, KEY30, KEY31, KEY32, KEY33, KEY34, KEY35, KEY4, KEY5, KEY6, KEY7, KEY8, KEY9: footprint key-switches:MX_switch_Gateron_hotswap_double_sided_A -> key-switches:MX_switch_THT_hotswap_double_sided_A

Commit message: Update
Parts:
- removed J3: Conn_01x06, Connector_PinHeader_2.54mm:PinHeader_1x06_P2.54mm_Vertical, symbol Connector_Generic:Conn_01x06
- removed J4: Conn_01x04, Connector_PinHeader_2.54mm:PinHeader_1x04_P2.54mm_Vertical, symbol Connector_Generic:Conn_01x04
- removed LD1: LED, LED_SMD:LED_0603_1608Metric, symbol Device:LED
- removed R2: 1k, Resistor_SMD:R_0603_1608Metric, symbol Device:R
- removed TP1, TP10, TP11, TP12, TP13, TP14, TP2, TP3, TP4, TP5, TP6, TP7, TP8, TP9: TestPoint, TestPoint:TestPoint_Pad_D2.5mm, symbol Connector:TestPoint
- added H1, H10, H11, H12, H13, H2, H3, H4, H5, H6, H7, H8, H9: MountingHole, MountingHole:MountingHole_2.2mm_M2, symbol Mechanical:MountingHole
- added J4: Conn_01x08, Connector_PinSocket_2.54mm:PinSocket_1x08_P2.54mm_Vertical, symbol Connector_Generic:Conn_01x08
- added SW2: RESET, Button_Switch_SMD:SW_SPST_TL3342, symbol Switch:SW_Push
- added SW4: SW_2P2T, ErgoSNM_Keybaord:MSK-23D20-T, symbol ErgoSNM_Keybaord_Library:SW_2P2T
- added TRRS2: PJ-393_TRRS_8P, ErgoSNM_Keybaord:PJ-393, symbol ErgoSNM_Keybaord_Library:PJ-393_TRRS_8P
- D1, D18, D35: footprint Diode_SMD:D_0603_1608Metric -> Diode_SMD:D_SOD-123
- D10: renamed from D30; footprint Diode_SMD:D_0603_1608Metric -> Diode_SMD:D_SOD-123
- D11: renamed from D3; footprint Diode_SMD:D_0603_1608Metric -> Diode_SMD:D_SOD-123
- D12: renamed from D10; footprint Diode_SMD:D_0603_1608Metric -> Diode_SMD:D_SOD-123
- D13: renamed from D17; footprint Diode_SMD:D_0603_1608Metric -> Diode_SMD:D_SOD-123
- D14: renamed from D24; footprint Diode_SMD:D_0603_1608Metric -> Diode_SMD:D_SOD-123
- D15: renamed from D31; footprint Diode_SMD:D_0603_1608Metric -> Diode_SMD:D_SOD-123
- D16: renamed from D4; footprint Diode_SMD:D_0603_1608Metric -> Diode_SMD:D_SOD-123
- D17: renamed from D11; footprint Diode_SMD:D_0603_1608Metric -> Diode_SMD:D_SOD-123
- D19: renamed from D25; footprint Diode_SMD:D_0603_1608Metric -> Diode_SMD:D_SOD-123
- D2: renamed from D8; footprint Diode_SMD:D_0603_1608Metric -> Diode_SMD:D_SOD-123
- D20: renamed from D32; footprint Diode_SMD:D_0603_1608Metric -> Diode_SMD:D_SOD-123
- D21: renamed from D5; footprint Diode_SMD:D_0603_1608Metric -> Diode_SMD:D_SOD-123
- D22: renamed from D12; footprint Diode_SMD:D_0603_1608Metric -> Diode_SMD:D_SOD-123
- D23: renamed from D19; footprint Diode_SMD:D_0603_1608Metric -> Diode_SMD:D_SOD-123
- D24: renamed from D26; footprint Diode_SMD:D_0603_1608Metric -> Diode_SMD:D_SOD-123
- D25: renamed from D33; footprint Diode_SMD:D_0603_1608Metric -> Diode_SMD:D_SOD-123
- D26: renamed from D6; footprint Diode_SMD:D_0603_1608Metric -> Diode_SMD:D_SOD-123
- D27: renamed from D13; footprint Diode_SMD:D_0603_1608Metric -> Diode_SMD:D_SOD-123
- D28: renamed from D20; footprint Diode_SMD:D_0603_1608Metric -> Diode_SMD:D_SOD-123
- D29: renamed from D27; footprint Diode_SMD:D_0603_1608Metric -> Diode_SMD:D_SOD-123
- D3: renamed from D15; footprint Diode_SMD:D_0603_1608Metric -> Diode_SMD:D_SOD-123
- D30: renamed from D34; footprint Diode_SMD:D_0603_1608Metric -> Diode_SMD:D_SOD-123
- D31: renamed from D7; footprint Diode_SMD:D_0603_1608Metric -> Diode_SMD:D_SOD-123
- D32: renamed from D14; footprint Diode_SMD:D_0603_1608Metric -> Diode_SMD:D_SOD-123
- D33: renamed from D21; footprint Diode_SMD:D_0603_1608Metric -> Diode_SMD:D_SOD-123
- D34: renamed from D28; footprint Diode_SMD:D_0603_1608Metric -> Diode_SMD:D_SOD-123
- D4: renamed from D22; footprint Diode_SMD:D_0603_1608Metric -> Diode_SMD:D_SOD-123
- D5: renamed from D29; footprint Diode_SMD:D_0603_1608Metric -> Diode_SMD:D_SOD-123
- D6: renamed from D2; footprint Diode_SMD:D_0603_1608Metric -> Diode_SMD:D_SOD-123
- D7: renamed from D9; footprint Diode_SMD:D_0603_1608Metric -> Diode_SMD:D_SOD-123
- D8: renamed from D16; footprint Diode_SMD:D_0603_1608Metric -> Diode_SMD:D_SOD-123
- D9: renamed from D23; footprint Diode_SMD:D_0603_1608Metric -> Diode_SMD:D_SOD-123
- SW1: footprint Button_Switch_SMD:SW_Push_1P1T_NO_6x6mm_H9.5mm -> Button_Switch_SMD:SW_SPST_TL3342
- renumbered J6 to J3, J7 to J6, KEY30 to KEY10, KEY3 to KEY11, KEY10 to KEY12, KEY17 to KEY13, KEY24 to KEY14, KEY31 to KEY15, KEY4 to KEY16, KEY11 to KEY17, KEY25 to KEY19, KEY8 to KEY2, KEY32 to KEY20, KEY5 to KEY21, KEY12 to KEY22, KEY19 to KEY23, KEY26 to KEY24, KEY33 to KEY25, KEY6 to KEY26, KEY13 to KEY27, KEY20 to KEY28, KEY27 to KEY29, KEY15 to KEY3, KEY34 to KEY30, KEY7 to KEY31, KEY14 to KEY32, KEY21 to KEY33, KEY28 to KEY34, KEY22 to KEY4, KEY29 to KEY5, KEY2 to KEY6, KEY9 to KEY7, KEY16 to KEY8, KEY23 to KEY9, R3 to R2, R4 to R3, SW2 to SW3
Connections:
- net SDA is gone; now on net ENC_B: J1.6 (Pin_6), R3.1, TRRS1.2 (R1a)
- net +BATT: now also SW3.2, SW4.2; no longer SW3.5
- net COL_6: now also J4.8 (Pin_8)
- net CS: now also J4.3 (Pin_3)
- net ENC_B: now also J4.7 (Pin_7), TRRS2.2 (R1a); no longer J1.7 (Pin_7), R2.2, TRRS1.3 (R2a)
- net GND: now also J4.2 (Pin_2), SW2.2, TRRS2.1 (Ta)
- net MISO: now also J4.5 (Pin_5)
- net MOSI: now also J4.4 (Pin_4)
- net RESET: now also SW2.1
- net SCLK: now also J4.6 (Pin_6)
- net VCC: now also J4.1 (Pin_1), TRRS2.8 (Sa)
- net at SW3.1: now also J3.2 (Pin_2), SW4.1
- net at SW3.4: no longer J3.2 (Pin_2)
- new net SCL: J1.7 (Pin_7), R2.2, TRRS1.3 (R2a), TRRS2.3 (R2a)
- no-connect marks 7 -> 12
Other:
- moved on the sheet: J1, J2, J3, J5, J6, R1, R2, R3, SW1, SW3, TRRS1
