File: ErgoSNM_Keyboard/rev1/ErgoSNM_keyboard.kicad_sch (KiCad schematic)
At the start: 98 parts, among them J1 Conn_01x13, J2 Conn_01x13, J3 Conn_01x03, J4 Conn_01x08, J5 Conn_01x07, J6 Conn_01x07, SW1 RESET, SW2 RESET, SW3 SW_2P2T, SW4 SW_2P2T

Commit message: Update `Rev 1.1`
Parts:
- TRRS1, TRRS2: footprint ErgoSNM_Keybaord:PJ-393 -> ErgoSNM_Keyboard:PJ-393 8P TRRS; symbol ErgoSNM_Keybaord_Library:PJ-393_TRRS_8P -> ErgoSNM_Keyboard_Library:PJ-393_TRRS_8P
Connections:
- net ENC_B: now also TRRS1.R1, TRRS2.R1; no longer TRRS1.2 (R1a), TRRS2.2 (R1a)
- net GND: now also TRRS1.T, TRRS2.T; no longer TRRS1.1 (Ta), TRRS2.1 (Ta)
- net SCL: now also TRRS1.R2, TRRS2.R2; no longer TRRS1.3 (R2a), TRRS2.3 (R2a)
- net VCC: now also TRRS1.S, TRRS2.S; no longer TRRS1.8 (Sa), TRRS2.8 (Sa)
Other:
- moved on the sheet: R2, R3
