File: ErgoSNM_Keyboard/rev3/left/mcu.kicad_sch (KiCad schematic)
At the start: 8 parts, among them U2 E73-2G4M08S1C

Commit message: Update submodule
Update submodule

Update switch footprint
Parts:
- renumbered U2 to U3
Changed lines of the file:
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@@
       (project "ErgoSNM_v3_left"
         (path "/94fd6fa5-abea-4c62-b80d-3b080722228a/55bd3253-f9d8-4021-ab54-3edc1cd235a5"
-          (reference "#PWR0105") (unit 1)
+          (reference "#PWR026") (unit 1)
         )
       )
@@
         )
         (path "/94fd6fa5-abea-4c62-b80d-3b080722228a/55bd3253-f9d8-4021-ab54-3edc1cd235a5"
-          (reference "#PWR0106") (unit 1)
+          (reference "#PWR024") (unit 1)
         )
       )
@@
         )
         (path "/94fd6fa5-abea-4c62-b80d-3b080722228a/55bd3253-f9d8-4021-ab54-3edc1cd235a5"
-          (reference "#PWR0103") (unit 1)
+          (reference "#PWR030") (unit 1)
         )
       )
@@
   (symbol (lib_id "ErgoSNM_Keyboard_Library:E73-2G4M08S1C") (at 128.27 110.49 0) (unit 1)
     (in_bom yes) (on_board yes) (dnp no) (fields_autoplaced)
-    (property "Reference" "U2" (at 133.0041 146.05 0)
+    (property "Reference" "U3" (at 133.0041 146.05 0)
       (effects (font (size 1.27 1.27)) (justify left))
     )
@@
       (project "ErgoSNM_v3_left"
         (path "/94fd6fa5-abea-4c62-b80d-3b080722228a/55bd3253-f9d8-4021-ab54-3edc1cd235a5"
-          (reference "U2") (unit 1)
+          (reference "U3") (unit 1)
         )
       )
@@
       (project "ErgoSNM_v3_left"
         (path "/94fd6fa5-abea-4c62-b80d-3b080722228a/55bd3253-f9d8-4021-ab54-3edc1cd235a5"
-          (reference "#PWR0102") (unit 1)
+          (reference "#PWR028") (unit 1)
         )
       )
@@
         )
         (path "/94fd6fa5-abea-4c62-b80d-3b080722228a/55bd3253-f9d8-4021-ab54-3edc1cd235a5"
-          (reference "SW3") (unit 1)
+          (reference "SW2") (unit 1)
         )
       )
@@
       (project "ErgoSNM_v3_left"
         (path "/94fd6fa5-abea-4c62-b80d-3b080722228a/55bd3253-f9d8-4021-ab54-3edc1cd235a5"
-          (reference "#PWR0108") (unit 1)
+          (reference "#PWR029") (unit 1)
         )
       )
@@
       (project "ErgoSNM_v3_left"
         (path "/94fd6fa5-abea-4c62-b80d-3b080722228a/55bd3253-f9d8-4021-ab54-3edc1cd235a5"
-          (reference "C3") (unit 1)
+          (reference "C5") (unit 1)
         )
       )
@@
       (project "ErgoSNM_v3_left"
         (path "/94fd6fa5-abea-4c62-b80d-3b080722228a/55bd3253-f9d8-4021-ab54-3edc1cd235a5"
-          (reference "#PWR0104") (unit 1)
+          (reference "#PWR031") (unit 1)
         )
       )
@@
         )
         (path "/94fd6fa5-abea-4c62-b80d-3b080722228a/55bd3253-f9d8-4021-ab54-3edc1cd235a5"
-          (reference "#PWR0107") (unit 1)
+          (reference "#PWR025") (unit 1)
         )
       )
@@
         )
         (path "/94fd6fa5-abea-4c62-b80d-3b080722228a/55bd3253-f9d8-4021-ab54-3edc1cd235a5"
-          (reference "#PWR0101") (unit 1)
+          (reference "#PWR027") (unit 1)
         )
       )
@@
       (project "ErgoSNM_v3_left"
         (path "/94fd6fa5-abea-4c62-b80d-3b080722228a/55bd3253-f9d8-4021-ab54-3edc1cd235a5"
-          (reference "C4") (unit 1)
-        )
-      )
+          (reference "C6") (unit 1)
+        )
+      )
