File: ErgoSNM_Keyboard/rev3/right/key_matrix.kicad_sch (KiCad schematic)
At the start: 58 parts

Commit message: Update submodule
Update submodule

Update switch footprint
Parts:
- renumbered D26 to D10, D3 to D11, D9 to D12, D15 to D13, D21 to D14, D27 to D15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
