File: ErgoSNM_Keyboard/rev3/right/mcu.kicad_sch (KiCad schematic)
At the start: 8 parts, among them U2 E73-2G4M08S1C

Commit message: Add LDO for USB
Changed lines of the file:
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@@
     (stroke (width 0) (type default))
-  )
-  (text_box "Power Mode:\n1. Reg0 DC/DC & LDO disable: JP 1-2 3, L DNI\n2. Reg0 DC/DC enable: JP 1 2-3, L 10uH"
-    (at 99.06 19.05 0) (size 50.8 7.62)
-    (stroke (width 0) (type default))
-    (fill (type none))
-    (effects (font (size 1.27 1.27)) (justify left top))
   )
   (label "VBUS" (at 132.08 71.12 270) (fields_autoplaced)

Commit message: Update submodule
Update submodule

Update switch footprint
Parts:
- renumbered U2 to U3
Connections:
- no-connect marks 0 -> 6
Changed lines of the file:
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@@
   (junction (at 138.43 50.8) (diameter 0) (color 0 0 0 0)
   )
+  (no_connect (at 144.78 115.57))
+  (no_connect (at 144.78 125.73))
+  (no_connect (at 144.78 100.33))
+  (no_connect (at 144.78 118.11))
+  (no_connect (at 144.78 110.49))
+  (no_connect (at 144.78 92.71))
   (wire (pts (xy 77.47 99.06) (xy 77.47 96.52))
     (stroke (width 0) (type default))
@@
     (stroke (width 0) (type default))
   )
-  (wire (pts (xy 104.14 121.92) (xy 110.49 121.92))
-    (stroke (width 0) (type default))
-  )
   (wire (pts (xy 119.38 52.07) (xy 119.38 50.8))
     (stroke (width 0) (type default))
@@
     (stroke (width 0) (type default))
   )
-  (wire (pts (xy 85.09 124.46) (xy 110.49 124.46))
-    (stroke (width 0) (type default))
-  )
   (wire (pts (xy 44.45 85.09) (xy 44.45 83.82))
     (stroke (width 0) (type default))
   )
-  (wire (pts (xy 104.14 119.38) (xy 110.49 119.38))
-    (stroke (width 0) (type default))
-  )
   (wire (pts (xy 82.55 96.52) (xy 77.47 96.52))
     (stroke (width 0) (type default))
   )
-  (wire (pts (xy 168.91 113.03) (xy 144.78 113.03))
-    (stroke (width 0) (type default))
-  )
   (wire (pts (xy 138.43 46.99) (xy 138.43 50.8))
     (stroke (width 0) (type default))
@@
     (stroke (width 0) (type default))
   )
-  (wire (pts (xy 168.91 95.25) (xy 144.78 95.25))
-    (stroke (width 0) (type default))
-  )
   (wire (pts (xy 129.54 71.12) (xy 129.54 77.47))
     (stroke (width 0) (type default))
@@
   )
   (wire (pts (xy 119.38 46.99) (xy 119.38 50.8))
-    (stroke (width 0) (type default))
-  )
-  (wire (pts (xy 85.09 129.54) (xy 110.49 129.54))
-    (stroke (width 0) (type default))
-  )
-  (wire (pts (xy 85.09 127) (xy 110.49 127))
     (stroke (width 0) (type default))
   )
@@
     )
   )
-  (global_label "PMW3360_Motion" (shape input) (at 85.09 124.46 180) (fields_autoplaced)
-    (effects (font (size 1.27 1.27)) (justify right))
-    (property "Intersheetrefs" "${INTERSHEET_REFS}" (at 65.8975 124.46 0)
+  (global_label "PMW3360_Motion" (shape input) (at 110.49 124.46 180) (fields_autoplaced)
+    (effects (font (size 1.27 1.27)) (justify right))
+    (property "Intersheetrefs" "${INTERSHEET_REFS}" (at 91.2975 124.46 0)
       (effects (font (size 1.27 1.27)) (justify right) hide)
     )
@@
     )
   )
-  (global_label "PMW3360_SPI_MOSI" (shape input) (at 85.09 129.54 180) (fields_autoplaced)
-    (effects (font (size 1.27 1.27)) (justify right))
-    (property "Intersheetrefs" "${INTERSHEET_REFS}" (at 63.4783 129.54 0)
+  (global_label "PMW3360_SPI_MOSI" (shape input) (at 110.49 129.54 180) (fields_autoplaced)
+    (effects (font (size 1.27 1.27)) (justify right))
+    (property "Intersheetrefs" "${INTERSHEET_REFS}" (at 88.8783 129.54 0)
       (effects (font (size 1.27 1.27)) (justify right) hide)
     )
@@
     )
   )
-  (global_label "PMW3360_SPI_CS" (shape input) (at 85.09 127 180) (fields_autoplaced)
-    (effects (font (size 1.27 1.27)) (justify right))
-    (property "Intersheetrefs" "${INTERSHEET_REFS}" (at 65.595 127 0)
+  (global_label "PMW3360_SPI_CS" (shape input) (at 110.49 127 180) (fields_autoplaced)
+    (effects (font (size 1.27 1.27)) (justify right))
+    (property "Intersheetrefs" "${INTERSHEET_REFS}" (at 90.995 127 0)
       (effects (font (size 1.27 1.27)) (justify right) hide)
     )
@@
     )
   )
-  (global_label "PMW3360_SPI_SCLK" (shape input) (at 168.91 113.03 0) (fields_autoplaced)
-    (effects (font (size 1.27 1.27)) (justify left))
-    (property "Intersheetrefs" "${INTERSHEET_REFS}" (at 190.7031 113.03 0)
+  (global_label "PMW3360_SPI_SCLK" (shape input) (at 144.78 113.03 0) (fields_autoplaced)
+    (effects (font (size 1.27 1.27)) (justify left))
+    (property "Intersheetrefs" "${INTERSHEET_REFS}" (at 166.5731 113.03 0)
       (effects (font (size 1.27 1.27)) (justify left) hide)
     )
@@
     )
   )
-  (global_label "QMK_UART_Rx" (shape input) (at 104.14 119.38 180) (fields_autoplaced)
-    (effects (font (size 1.27 1.27)) (justify right))
-    (property "Intersheetrefs" "${INTERSHEET_REFS}" (at 88.2129 119.38 0)
+  (global_label "QMK_UART_Rx" (shape input) (at 110.49 119.38 180) (fields_autoplaced)
+    (effects (font (size 1.27 1.27)) (justify right))
+    (property "Intersheetrefs" "${INTERSHEET_REFS}" (at 94.5629 119.38 0)
       (effects (font (size 1.27 1.27)) (justify right) hide)
     )
@@
     )
   )
-  (global_label "PMW3360_SPI_MISO" (shape input) (at 168.91 95.25 0) (fields_autoplaced)
-    (effects (font (size 1.27 1.27)) (justify left))
-    (property "Intersheetrefs" "${INTERSHEET_REFS}" (at 190.5217 95.25 0)
+  (global_label "PMW3360_SPI_MISO" (shape input) (at 144.78 95.25 0) (fields_autoplaced)
+    (effects (font (size 1.27 1.27)) (justify left))
+    (property "Intersheetrefs" "${INTERSHEET_REFS}" (at 166.3917 95.25 0)
       (effects (font (size 1.27 1.27)) (justify left) hide)
     )
@@
     )
   )
-  (global_label "QMK_UART_Tx" (shape input) (at 104.14 121.92 180) (fields_autoplaced)
-    (effects (font (size 1.27 1.27)) (justify right))
-    (property "Intersheetrefs" "${INTERSHEET_REFS}" (at 88.5153 121.92 0)
+  (global_label "QMK_UART_Tx" (shape input) (at 110.49 121.92 180) (fields_autoplaced)
+    (effects (font (size 1.27 1.27)) (justify right))
+    (property "Intersheetrefs" "${INTERSHEET_REFS}" (at 94.8653 121.92 0)
       (effects (font (size 1.27 1.27)) (justify right) hide)
     )
@@
       (project "ErgoSNM_v3_right"
         (path "/94fd6fa5-abea-4c62-b80d-3b080722228a/4dfe88da-5f2a-417e-8535-56638ceff4df"
-          (reference "#PWR024") (unit 1)
+          (reference "#PWR027") (unit 1)
         )
       )
@@
         )
         (path "/94fd6fa5-abea-4c62-b80d-3b080722228a/4dfe88da-5f2a-417e-8535-56638ceff4df"
-          (reference "#PWR022") (unit 1)
+          (reference "#PWR025") (unit 1)
         )
       )
@@
         )
         (path "/94fd6fa5-abea-4c62-b80d-3b080722228a/4dfe88da-5f2a-417e-8535-56638ceff4df"
-          (reference "#PWR019") (unit 1)
+          (reference "#PWR031") (unit 1)
         )
       )
@@
   (symbol (lib_id "ErgoSNM_Keyboard_Library:E73-2G4M08S1C") (at 128.27 110.49 0) (unit 1)
     (in_bom yes) (on_board yes) (dnp no) (fields_autoplaced)
-    (property "Reference" "U2" (at 133.0041 146.05 0)
+    (property "Reference" "U3" (at 133.0041 146.05 0)
       (effects (font (size 1.27 1.27)) (justify left))
     )
@@
       (project "ErgoSNM_v3_right"
         (path "/94fd6fa5-abea-4c62-b80d-3b080722228a/4dfe88da-5f2a-417e-8535-56638ceff4df"
-          (reference "U2") (unit 1)
+          (reference "U3") (unit 1)
         )
       )
@@
       (project "ErgoSNM_v3_right"
         (path "/94fd6fa5-abea-4c62-b80d-3b080722228a/4dfe88da-5f2a-417e-8535-56638ceff4df"
-          (reference "#PWR020") (unit 1)
+          (reference "#PWR029") (unit 1)
         )
       )
@@
       (project "ErgoSNM_v3_right"
         (path "/94fd6fa5-abea-4c62-b80d-3b080722228a/4dfe88da-5f2a-417e-8535-56638ceff4df"
-          (reference "C4") (unit 1)
+          (reference "C8") (unit 1)
         )
       )
@@
       (project "ErgoSNM_v3_right"
         (path "/94fd6fa5-abea-4c62-b80d-3b080722228a/4dfe88da-5f2a-417e-8535-56638ceff4df"
-          (reference "C3") (unit 1)
+          (reference "C7") (unit 1)
         )
       )
@@
       (project "ErgoSNM_v3_right"
         (path "/94fd6fa5-abea-4c62-b80d-3b080722228a/4dfe88da-5f2a-417e-8535-56638ceff4df"
-          (reference "#PWR025") (unit 1)
+          (reference "#PWR030") (unit 1)
         )
       )
@@
       (project "ErgoSNM_v3_right"
         (path "/94fd6fa5-abea-4c62-b80d-3b080722228a/4dfe88da-5f2a-417e-8535-56638ceff4df"
-          (reference "#PWR021") (unit 1)
+          (reference "#PWR032") (unit 1)
         )
       )
@@
         )
         (path "/94fd6fa5-abea-4c62-b80d-3b080722228a/4dfe88da-5f2a-417e-8535-56638ceff4df"
-          (reference "#PWR023") (unit 1)
+          (reference "#PWR026") (unit 1)
         )
       )
@@
         )
         (path "/94fd6fa5-abea-4c62-b80d-3b080722228a/4dfe88da-5f2a-417e-8535-56638ceff4df"
-          (reference "#PWR018") (unit 1)
-        )
-      )
+          (reference "#PWR028") (unit 1)
+        )
+      )
