File: ErgoSNM_Keyboard/rev2/left/RP2040.kicad_sch (KiCad schematic)
At the start: 26 parts, among them SW1 BOOT, SW2 RESET, U3 RP2040, U4 W25Q128JVS, Y1 12MHz

Commit message: Update rev2
Parts:
- removed JP1: SolderJumper_3_Bridged12, Jumper:SolderJumper-3_P1.3mm_Bridged12_Pad1.0x1.5mm_NumberLabels, symbol Jumper:SolderJumper_3_Bridged12
- added TP3, TP4: TestPoint, TestPoint:TestPoint_Pad_D2.5mm, symbol Connector:TestPoint
- renumbered C11 to C10, C12 to C11, C13 to C12, C14 to C13, C15 to C14, C17 to C16, C4 to C3, C5 to C4, C6 to C5, C7 to C6, C8 to C7, C9 to C8, R5 to R3, R6 to R4, R7 to R5, R8 to R6, R9 to R7, R10 to R8
Connections:
- net Handedness is gone; now on net MISO: U3.31 (GPIO20)
- net RGB_LED_DATA_3V3 is gone; now on net Encoder_A: U3.30 (GPIO19)
- net +3V3: now also U3.18 (GPIO15)
- net COL_0: now also U3.14 (GPIO11); no longer U3.4 (GPIO2)
- net COL_1: now also U3.13 (GPIO10); no longer U3.5 (GPIO3)
- net COL_2: now also U3.12 (GPIO9); no longer U3.6 (GPIO4)
- net COL_3: now also U3.8 (GPIO6); no longer U3.7 (GPIO5)
- net COL_4: now also U3.7 (GPIO5); no longer U3.3 (GPIO1)
- net COL_5: now also U3.6 (GPIO4); no longer U3.8 (GPIO6)
- net COL_6: now also U3.28 (GPIO17); no longer U3.35 (GPIO23)
- net CS: now also U3.32 (GPIO21); no longer U3.12 (GPIO9)
- net Encoder_A: no longer U3.29 (GPIO18)
- net Encoder_B: now also U3.29 (GPIO18); no longer U3.28 (GPIO17)
- net MISO: no longer U3.11 (GPIO8)
- net MOSI: now also U3.35 (GPIO23); no longer U3.14 (GPIO11)
- net ROW_0: now also U3.40 (GPIO28_ADC2); no longer U3.36 (GPIO24)
- net ROW_1: now also U3.39 (GPIO27_ADC1); no longer U3.37 (GPIO25)
- net ROW_3: now also U3.37 (GPIO25); no longer U3.39 (GPIO27_ADC1)
- net ROW_4: now also U3.36 (GPIO24); no longer U3.40 (GPIO28_ADC2)
- net SCLK: now also U3.34 (GPIO22); no longer U3.13 (GPIO10)
- net SERIAL: now also U3.5 (GPIO3); no longer U3.15 (GPIO12)
- net SWCLK: now also TP3.1
- net SWDIO: now also TP4.1

Commit message: Update BOM, net, placement, etc.
Parts:
- added R4: 5.1k, Resistor_SMD:R_0402_1005Metric, symbol Device:R
- C10: renamed from C8; JLCPCB Part # C307331 -> (none); LCSC (none) -> C307331
- C11: renamed from C10; JLCPCB Part # C307331 -> (none); LCSC (none) -> C307331
- C12: renamed from C11; JLCPCB Part # C307331 -> (none); LCSC (none) -> C307331
- C13: renamed from C12; JLCPCB Part # C307331 -> (none); LCSC (none) -> C307331
- C14: renamed from C13; JLCPCB Part # C307331 -> (none); LCSC (none) -> C307331
- C15: renamed from C14; JLCPCB Part # C307331 -> (none); LCSC (none) -> C307331
- C3: renamed from C16; JLCPCB Part # C307331 -> (none); LCSC (none) -> C307331
- C4: renamed from C5; JLCPCB Part # C1554 -> (none); LCSC (none) -> C1554
- C5: renamed from C6; JLCPCB Part # C1554 -> (none); LCSC (none) -> C1554
- C6: renamed from C3; JLCPCB Part # C307331 -> (none); LCSC (none) -> C307331
- C7: JLCPCB Part # C307331 -> (none); LCSC (none) -> C307331
- C9: renamed from C4; JLCPCB Part # C307331 -> (none); LCSC (none) -> C307331
- C? (x2): JLCPCB Part # C52923 -> (none); LCSC (none) -> C52923
- R10: renamed from R8; JLCPCB Part # C25744 -> (none); LCSC (none) -> C25744
- R5: renamed from R3; JLCPCB Part # C25100 -> (none); LCSC (none) -> C25190; MFR. Part # 0402WGF270JTCE -> 0603WAF270JT5E
- R6: renamed from R4; JLCPCB Part # C25100 -> (none); LCSC (none) -> C25190; MFR. Part # 0402WGF270JTCE -> 0603WAF270JT5E
- R7: renamed from R6; JLCPCB Part # C11702 -> (none); LCSC (none) -> C11702
- R8: renamed from R7; JLCPCB Part # C25744 -> (none); LCSC (none) -> C25744
- R9: renamed from R5; JLCPCB Part # C11702 -> (none); LCSC (none) -> C11702
- SW1, SW2: JLCPCB Part # C231329 -> (none); LCSC (none) -> C318884; MFR. Part # B3U-1000P -> TS-1187A-B-A-B
- TP5: renamed from TP3; now left out of the parts list
- TP6: renamed from TP4; now left out of the parts list
- U3: renamed from U4; LCSC (none) -> C97521; MFR. Part # (none) -> W25Q128JVSIQ
- U4: renamed from U3; JLCPCB Part # C2040 -> (none); LCSC (none) -> C2040
- Y1: JLCPCB Part # C9002 -> (none); LCSC (none) -> C9002
Connections:
- net MOSI is gone; now on net Encoder_A: U4.35 (GPIO23)
- net SCLK is gone; now on net COL_6: U4.34 (GPIO22)
- net +3V3: now also R4.2
- net COL_6: no longer U4.28 (GPIO17)
- net Encoder_A: no longer U4.30 (GPIO19)
- net SERIAL: now also U4.2 (GPIO0), R4.1; no longer U4.5 (GPIO3)
- net CS renamed COL_7
- net MISO renamed ROW_5
- new net STATE_LED: U4.28 (GPIO17)
- no-connect marks 0 -> 11
Other:
- note added: "By default, high is left"
- note added: "Flash"
- note added: "MISO"
- note added: "MOSI"
- note added: "SCLK"
- note added: "~{CS}"
- moved on the sheet: C10, C11, C12, C13, C14, C15, C3, C6, C7, C9, C?, R10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

Commit message: Change license to CERN-OHL-P v2
Parts:
- gave numbers to parts that had none: 2
