File: ErgoSNM_Keyboard/rev2/left/key_matrix.kicad_sch (KiCad schematic)
At the start: 60 parts, among them J3 Conn_01x08, J4 Conn_01x08

Commit message: Update rev2
Parts:
- J3: footprint Connector_PinSocket_2.00mm:PinSocket_1x08_P2.00mm_Vertical -> Connector_PinSocket_2.00mm:PinSocket_2x04_P2.00mm_Vertical; symbol Connector_Generic:Conn_01x08 -> Connector_Generic:Conn_02x04_Odd_Even
- J4: footprint ErgoSNM_Keyboard:FPC_8P_0.5mm -> ErgoSNM_Keyboard:FPC_8P_1.0mm
Connections:
- net COL_5: now also KEY29.1; no longer KEY29.2
- net ROW_0: now also J4.3 (Pin_3); no longer J4.7 (Pin_7)
- net ROW_1: now also J4.4 (Pin_4); no longer J4.6 (Pin_6)
- net ROW_3: now also J4.6 (Pin_6); no longer J4.4 (Pin_4)
- net ROW_4: now also J4.7 (Pin_7); no longer J4.3 (Pin_3)
- net at D29.2 (A): now also KEY29.2; no longer KEY29.1
Other:
- moved on the sheet: J3, KEY29
Changed lines of the file:
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@@
     (stroke (width 0) (type default) (color 0 0 0 0))
   )
-  (global_label "ROW_0" (shape input) (at 251.46 71.12 180) (fields_autoplaced)
-    (effects (font (size 1.27 1.27)) (justify right))
-    (property "Intersheet References" "${INTERSHEET_REFS}" (id 0) (at 242.8179 71.0406 0)
-      (effects (font (size 1.27 1.27)) (justify right) hide)
-    )
-  )
   (global_label "ROW_4" (shape input) (at 92.71 139.7 180) (fields_autoplaced)
     (effects (font (size 1.27 1.27)) (justify right))
@@
     )
   )
-  (global_label "ROW_1" (shape input) (at 251.46 73.66 180) (fields_autoplaced)
+  (global_label "ROW_3" (shape input) (at 264.16 76.2 0) (fields_autoplaced)
+    (effects (font (size 1.27 1.27)) (justify left))
+    (property "Intersheet References" "${INTERSHEET_REFS}" (id 0) (at 272.8021 76.2794 0)
+      (effects (font (size 1.27 1.27)) (justify left) hide)
+    )
+  )
+  (global_label "ROW_4" (shape input) (at 251.46 78.74 180) (fields_autoplaced)
+    (effects (font (size 1.27 1.27)) (justify right))
+    (property "Intersheet References" "${INTERSHEET_REFS}" (id 0) (at 242.8179 78.6606 0)
+      (effects (font (size 1.27 1.27)) (justify right) hide)
+    )
+  )
+  (global_label "COL_6" (shape input) (at 251.46 71.12 180) (fields_autoplaced)
+    (effects (font (size 1.27 1.27)) (justify right))
+    (property "Intersheet References" "${INTERSHEET_REFS}" (id 0) (at 243.2412 71.0406 0)
+      (effects (font (size 1.27 1.27)) (justify right) hide)
+    )
+  )
+  (global_label "ROW_0" (shape input) (at 251.46 73.66 180) (fields_autoplaced)
     (effects (font (size 1.27 1.27)) (justify right))
     (property "Intersheet References" "${INTERSHEET_REFS}" (id 0) (at 242.8179 73.5806 0)
@@
     )
   )
-  (global_label "ROW_4" (shape input) (at 251.46 81.28 180) (fields_autoplaced)
-    (effects (font (size 1.27 1.27)) (justify right))
-    (property "Intersheet References" "${INTERSHEET_REFS}" (id 0) (at 242.8179 81.2006 0)
-      (effects (font (size 1.27 1.27)) (justify right) hide)
-    )
-  )
   (global_label "ROW_2" (shape input) (at 237.49 100.33 180) (fields_autoplaced)
     (effects (font (size 1.27 1.27)) (justify right))
-    (property "Intersheet References" "${INTERSHEET_REFS}" (id 0) (at 228.8479 100.4094 0)
+    (property "Intersheet References" "${INTERSHEET_REFS}" (id 0) (at 228.8479 100.2506 0)
       (effects (font (size 1.27 1.27)) (justify right) hide)
     )
@@
     )
   )
+  (global_label "COL_5" (shape input) (at 264.16 71.12 0) (fields_autoplaced)
+    (effects (font (size 1.27 1.27)) (justify left))
+    (property "Intersheet References" "${INTERSHEET_REFS}" (id 0) (at 272.3788 71.1994 0)
+      (effects (font (size 1.27 1.27)) (justify left) hide)
+    )
+  )
   (global_label "ROW_1" (shape input) (at 92.71 82.55 180) (fields_autoplaced)
     (effects (font (size 1.27 1.27)) (justify right))
@@
     )
   )
-  (global_label "COL_5" (shape input) (at 251.46 68.58 180) (fields_autoplaced)
-    (effects (font (size 1.27 1.27)) (justify right))
-    (property "Intersheet References" "${INTERSHEET_REFS}" (id 0) (at 243.2412 68.5006 0)
-      (effects (font (size 1.27 1.27)) (justify right) hide)
-    )
-  )
-  (global_label "ROW_3" (shape input) (at 237.49 97.79 180) (fields_autoplaced)
-    (effects (font (size 1.27 1.27)) (justify right))
-    (property "Intersheet References" "${INTERSHEET_REFS}" (id 0) (at 228.8479 97.8694 0)
-      (effects (font (size 1.27 1.27)) (justify right) hide)
-    )
-  )
-  (global_label "ROW_1" (shape input) (at 237.49 102.87 180) (fields_autoplaced)
-    (effects (font (size 1.27 1.27)) (justify right))
-    (property "Intersheet References" "${INTERSHEET_REFS}" (id 0) (at 228.8479 102.9494 0)
+  (global_label "ROW_3" (shape input) (at 237.49 102.87 180) (fields_autoplaced)
+    (effects (font (size 1.27 1.27)) (justify right))
+    (property "Intersheet References" "${INTERSHEET_REFS}" (id 0) (at 228.8479 102.7906 0)
+      (effects (font (size 1.27 1.27)) (justify right) hide)
+    )
+  )
+  (global_label "ROW_1" (shape input) (at 237.49 97.79 180) (fields_autoplaced)
+    (effects (font (size 1.27 1.27)) (justify right))
+    (property "Intersheet References" "${INTERSHEET_REFS}" (id 0) (at 228.8479 97.7106 0)
       (effects (font (size 1.27 1.27)) (justify right) hide)
     )
@@
     )
   )
-  (global_label "COL_6" (shape input) (at 251.46 66.04 180) (fields_autoplaced)
-    (effects (font (size 1.27 1.27)) (justify right))
-    (property "Intersheet References" "${INTERSHEET_REFS}" (id 0) (at 243.2412 65.9606 0)
-      (effects (font (size 1.27 1.27)) (justify right) hide)
-    )
-  )
-  (global_label "ROW_0" (shape input) (at 237.49 105.41 180) (fields_autoplaced)
-    (effects (font (size 1.27 1.27)) (justify right))
-    (property "Intersheet References" "${INTERSHEET_REFS}" (id 0) (at 228.8479 105.4894 0)
+  (global_label "ROW_0" (shape input) (at 237.49 95.25 180) (fields_autoplaced)
+    (effects (font (size 1.27 1.27)) (justify right))
+    (property "Intersheet References" "${INTERSHEET_REFS}" (id 0) (at 228.8479 95.1706 0)
       (effects (font (size 1.27 1.27)) (justify right) hide)
     )
@@
     )
   )
-  (global_label "ROW_3" (shape input) (at 251.46 78.74 180) (fields_autoplaced)
-    (effects (font (size 1.27 1.27)) (justify right))
-    (property "Intersheet References" "${INTERSHEET_REFS}" (id 0) (at 242.8179 78.6606 0)
-      (effects (font (size 1.27 1.27)) (justify right) hide)
-    )
-  )
-  (global_label "ROW_4" (shape input) (at 237.49 95.25 180) (fields_autoplaced)
-    (effects (font (size 1.27 1.27)) (justify right))
-    (property "Intersheet References" "${INTERSHEET_REFS}" (id 0) (at 228.8479 95.3294 0)
+  (global_label "ROW_1" (shape input) (at 264.16 73.66 0) (fields_autoplaced)
+    (effects (font (size 1.27 1.27)) (justify left))
+    (property "Intersheet References" "${INTERSHEET_REFS}" (id 0) (at 272.8021 73.7394 0)
+      (effects (font (size 1.27 1.27)) (justify left) hide)
+    )
+  )
+  (global_label "ROW_4" (shape input) (at 237.49 105.41 180) (fields_autoplaced)
+    (effects (font (size 1.27 1.27)) (justify right))
+    (property "Intersheet References" "${INTERSHEET_REFS}" (id 0) (at 228.8479 105.3306 0)
       (effects (font (size 1.27 1.27)) (justify right) hide)
     )
@@
   (symbol (lib_id "power:GND") (at 251.46 107.95 0) (unit 1)
     (in_bom yes) (on_board yes)
-    (property "Reference" "#PWR042" (id 0) (at 251.46 114.3 0)
+    (property "Reference" "#PWR035" (id 0) (at 251.46 114.3 0)
       (effects (font (size 1.27 1.27)) hide)
     )
@@
     (pin "2")
   )
-  (symbol (lib_id "Connector_Generic:Conn_01x08") (at 256.54 73.66 0) (unit 1)
-    (in_bom yes) (on_board yes) (fields_autoplaced)
-    (property "Reference" "J3" (id 0) (at 259.08 73.6599 0)
+  (symbol (lib_id "Connector_Generic:Conn_02x04_Odd_Even") (at 256.54 73.66 0) (unit 1)
+    (in_bom yes) (on_board yes)
+    (property "Reference" "J3" (id 0) (at 256.54 66.04 0)
       (effects (font (size 1.27 1.27)) (justify left))
     )
-    (property "Value" "Conn_01x08" (id 1) (at 259.08 76.1999 0)
+    (property "Value" "Conn_01x08" (id 1) (at 252.73 67.31 0)
       (effects (font (size 1.27 1.27)) (justify left))
     )
-    (property "Footprint" "Connector_PinSocket_2.00mm:PinSocket_1x08_P2.00mm_Vertical" (id 2) (at 256.54 73.66 0)
+    (property "Footprint" "Connector_PinSocket_2.00mm:PinSocket_2x04_P2.00mm_Vertical" (id 2) (at 256.54 73.66 0)
       (effects (font (size 1.27 1.27)) hide)
     )
@@
       (effects (font (size 1.27 1.27)) (justify left))
     )
-    (property "Footprint" "ErgoSNM_Keyboard:FPC_8P_0.5mm" (id 2) (at 256.54 97.79 0)
+    (property "Footprint" "ErgoSNM_Keyboard:FPC_8P_1.0mm" (id 2) (at 256.54 97.79 0)
       (effects (font (size 1.27 1.27)) hide)
     )
@@
     (pin "2")
   )
-  (symbol (lib_id "Switch:SW_Push_45deg") (at 191.77 110.49 180) (unit 1)
-    (in_bom yes) (on_board yes)
-    (property "Reference" "KEY29" (id 0) (at 194.31 107.95 0))
-    (property "Value" "SW_Push_45deg" (id 1) (at 191.77 115.57 0)
+  (symbol (lib_id "Switch:SW_Push_45deg") (at 191.77 110.49 0) (unit 1)
+    (in_bom yes) (on_board yes)
+    (property "Reference" "KEY29" (id 0) (at 191.77 105.41 0))
+    (property "Value" "SW_Push_45deg" (id 1) (at 191.77 105.41 0)
       (effects (font (size 1.27 1.27)) hide)
     )
@@
     (pin "2")
   )
-  (symbol (lib_id "power:GND") (at 251.46 83.82 0) (unit 1)
-    (in_bom yes) (on_board yes)
-    (property "Reference" "#PWR041" (id 0) (at 251.46 90.17 0)
-      (effects (font (size 1.27 1.27)) hide)
-    )
-    (property "Value" "GND" (id 1) (at 251.46 87.63 0))
-    (property "Footprint" "" (id 2) (at 251.46 83.82 0)
-      (effects (font (size 1.27 1.27)) hide)
-    )
-    (property "Datasheet" "" (id 3) (at 251.46 83.82 0)
-      (effects (font (size 1.27 1.27)) hide)
-    )
+  (symbol (lib_id "power:GND") (at 264.16 78.74 0) (unit 1)
+    (in_bom yes) (on_board yes)
+    (property "Reference" "#PWR036" (id 0) (at 264.16 85.09 0)
+      (effects (font (size 1.27 1.27)) hide)
+    )
+    (property "Value" "GND" (id 1) (at 264.16 82.55 0))
+    (property "Footprint" "" (id 2) (at 264.16 78.74 0)
+      (effects (font (size 1.27 1.27)) hide)
+    )
+    (property "Datasheet" "" (id 3) (at 264.16 78.74 0)
+      (effects (font (size 1.27 1.27)) hide)
+    )

Commit message: Update BOM, net, placement, etc.
Parts:
- removed J3: Conn_01x08, Connector_PinSocket_2.00mm:PinSocket_2x04_P2.00mm_Vertical, symbol Connector_Generic:Conn_02x04_Odd_Even
- removed J4: Conn_01x08, ErgoSNM_Keyboard:FPC_8P_1.0mm, symbol Connector_Generic:Conn_01x08
- D1: LCSC (none) -> C81598; MFR. Part # (none) -> 1N4148W
- D10: renamed from D17; LCSC (none) -> C81598; MFR. Part # (none) -> 1N4148W
- D11: renamed from D22; LCSC (none) -> C81598; MFR. Part # (none) -> 1N4148W
- D12: renamed from D27; LCSC (none) -> C81598; MFR. Part # (none) -> 1N4148W
- D13: renamed from D3; LCSC (none) -> C81598; MFR. Part # (none) -> 1N4148W
- D14: renamed from D8; LCSC (none) -> C81598; MFR. Part # (none) -> 1N4148W
- D15: renamed from D13; LCSC (none) -> C81598; MFR. Part # (none) -> 1N4148W
- D16: renamed from D18; LCSC (none) -> C81598; MFR. Part # (none) -> 1N4148W
- D17: renamed from D23; LCSC (none) -> C81598; MFR. Part # (none) -> 1N4148W
- D18: renamed from D28; LCSC (none) -> C81598; MFR. Part # (none) -> 1N4148W
- D19: renamed from D4; LCSC (none) -> C81598; MFR. Part # (none) -> 1N4148W
- D2: renamed from D6; LCSC (none) -> C81598; MFR. Part # (none) -> 1N4148W
- D20: renamed from D9; LCSC (none) -> C81598; MFR. Part # (none) -> 1N4148W
- D21: renamed from D14; LCSC (none) -> C81598; MFR. Part # (none) -> 1N4148W
- D22: renamed from D19; LCSC (none) -> C81598; MFR. Part # (none) -> 1N4148W
- D23: renamed from D24; LCSC (none) -> C81598; MFR. Part # (none) -> 1N4148W
- D24: renamed from D29; LCSC (none) -> C81598; MFR. Part # (none) -> 1N4148W
- D25: renamed from D5; LCSC (none) -> C81598; MFR. Part # (none) -> 1N4148W
- D26: renamed from D10; LCSC (none) -> C81598; MFR. Part # (none) -> 1N4148W
- D27: renamed from D15; LCSC (none) -> C81598; MFR. Part # (none) -> 1N4148W
- D28: renamed from D20; LCSC (none) -> C81598; MFR. Part # (none) -> 1N4148W
- D29: renamed from D25; LCSC (none) -> C81598; MFR. Part # (none) -> 1N4148W
- D3: renamed from D11; LCSC (none) -> C81598; MFR. Part # (none) -> 1N4148W
- D4: renamed from D16; LCSC (none) -> C81598; MFR. Part # (none) -> 1N4148W
- D5: renamed from D21; LCSC (none) -> C81598; MFR. Part # (none) -> 1N4148W
- D6: renamed from D26; LCSC (none) -> C81598; MFR. Part # (none) -> 1N4148W
- D7: renamed from D2; LCSC (none) -> C81598; MFR. Part # (none) -> 1N4148W
- D8: renamed from D7; LCSC (none) -> C81598; MFR. Part # (none) -> 1N4148W
- D9: renamed from D12; LCSC (none) -> C81598; MFR. Part # (none) -> 1N4148W
- renumbered KEY17 to KEY10, KEY22 to KEY11, KEY27 to KEY12, KEY3 to KEY13, KEY8 to KEY14, KEY13 to KEY15, KEY18 to KEY16, KEY23 to KEY17, KEY28 to KEY18, KEY4 to KEY19, KEY6 to KEY2, KEY9 to KEY20, KEY14 to KEY21, KEY19 to KEY22, KEY24 to KEY23, KEY29 to KEY24, KEY5 to KEY25, KEY10 to KEY26, KEY15 to KEY27, KEY20 to KEY28, KEY25 to KEY29, KEY11 to KEY3, KEY16 to KEY4, KEY21 to KEY5, KEY26 to KEY6, KEY2 to KEY7, KEY7 to KEY8, KEY12 to KEY9
