File: ErgoSNM_Keyboard/rev3/receiver/receiver.kicad_pcb (KiCad board)
At the start: 2 copper layers, 45 x 17.8 mm, 33 parts, among them J1 Conn_01x13, J2 Conn_01x13, J3 Conn_01x04, J4 Conn_02x05_Counter_Clockwise, J5 Conn_01x04, SW1 RESET, U1 E73-2G4M08S1C, Y1 32.768kHz

Commit message: Change license to CERN-OHL-P v2
Parts:
- J2: moved to B.Cu
- J4: renamed from J1; moved to B.Cu
- turned J2 to -90 degrees
- turned J4 to -90 degrees
- renumbered H5 to H1, H8 to H10, H9 to H11, H10 to H12, H11 to H13, H12 to H14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
