File: ErgoSNM_Keyboard/rev4/core_board_mdbt50q/core_board_mdbt50q.kicad_pcb (KiCad board)
At the start: 2 copper layers, 50.8 x 36.2 mm, 54 parts, among them J1 USB_C_Receptacle_USB2.0, J2 USB_C_Receptacle_USB2.0, J3 Conn_01x30, J4 Conn_Batt, J5 Debug, SW1 SW_DPDT_x2, U1 MDBT50Q-1MV2, U2 SRV05-4, U3 TPS63020, U4 BQ24075RGT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

Commit message: feat: routed E73 core board
Other:
- board text added: "ErgoSNM"
