File: ErgoSNM_Keyboard/rev4/core_board_e73/power.kicad_sch (KiCad schematic)
At the start: 36 parts, among them J1 USB_C_Receptacle_USB2.0, J6 Conn_Batt, SW1 SW_SPDT, SW2 SW_SPDT, U2 USBLC6-2SC6, U3 BQ24075RGT, U4 TPS63900

Commit message: feat: update BOM
Parts:
- J6: Rotation Offset (none) -> 180
- R16: JLCPCB Part # C22765 -> C22809; MFR. Part # 0603WAF1201T5E -> 0603WAF1502T5E
- R19: JLCPCB Part # C22984 -> C4184; MFR. Part # 0603WAF3002T5E -> 0603WAF2002T5E
- SW1: now not fitted
- U2: Rotation Offset (none) -> 90
Changed lines of the file:
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@@
 			)
 		)
-		(property "JLCPCB Part #" "C22984"
+		(property "JLCPCB Part #" "C4184"
 			(at 264.16 81.28 0)
 			(effects
@@
 			)
 		)
-		(property "MFR. Part #" "0603WAF3002T5E"
+		(property "MFR. Part #" "0603WAF2002T5E"
 			(at 264.16 81.28 0)
 			(effects
@@
 			)
 		)
+		(property "Rotation Offset" "180"
+			(at 204.47 142.24 0)
+			(effects
+				(font
+					(size 1.27 1.27)
+				)
+				(hide yes)
+			)
+		)
 		(pin "2"
 		)
@@
 			)
 		)
-		(property "JLCPCB Part #" "C22765"
+		(property "JLCPCB Part #" "C22809"
 			(at 240.03 81.28 0)
 			(effects
@@
 			)
 		)
-		(property "MFR. Part #" "0603WAF1201T5E"
+		(property "MFR. Part #" "0603WAF1502T5E"
 			(at 240.03 81.28 0)
 			(effects
@@
 		(in_bom yes)
 		(on_board yes)
-		(dnp no)
+		(dnp yes)
 		(fields_autoplaced yes)
 		(property "Reference" "SW1"
@@
 			(at 92.71 142.24 0)
 			(effects
+				(font
+					(size 1.27 1.27)
+				)
+				(hide yes)
+			)
+		)
+		(property "Rotation Offset" "90"
+			(at 92.71 142.24 0)
+			(effects

Commit message: fix: add B5819 for battery reverse protection
Parts:
- added D1: B5819, Diode_SMD:D_SOD-323_HandSoldering, symbol Diode:1N5819WS
Connections:
- net VBATT_SRC: now also D1.1 (K); no longer R14.2, R15.2
- new net: D1.2 (A), R14.2, R15.2
Other:
- moved on the sheet: R14, R15
Changed lines of the file:
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@@
 	(text "2xAA Battery\nor\nLiPo Battery"
 		(exclude_from_sim no)
-		(at 146.05 60.96 0)
+		(at 137.16 60.96 0)
 		(effects
 			(font
@@
 	)
 	(junction
-		(at 156.21 58.42)
+		(at 60.96 142.24)
 		(diameter 0)
 		(color 0 0 0 0)
 	)
 	(junction
-		(at 60.96 142.24)
+		(at 175.26 58.42)
 		(diameter 0)
 		(color 0 0 0 0)
@@
 	)
 	(junction
-		(at 63.5 127)
+		(at 147.32 58.42)
 		(diameter 0)
 		(color 0 0 0 0)
 	)
 	(junction
-		(at 175.26 58.42)
+		(at 63.5 127)
 		(diameter 0)
 		(color 0 0 0 0)
@@
 	(wire
 		(pts
-			(xy 146.05 58.42) (xy 156.21 58.42)
+			(xy 137.16 58.42) (xy 147.32 58.42)
 		)
 		(stroke
@@
 	(wire
 		(pts
+			(xy 160.02 58.42) (xy 175.26 58.42)
+		)
+		(stroke
+			(width 0)
+			(type default)
+		)
+	)
+	(wire
+		(pts
 			(xy 99.06 144.78) (xy 97.79 144.78)
 		)
@@
 	(wire
 		(pts
+			(xy 147.32 58.42) (xy 152.4 58.42)
+		)
+		(stroke
+			(width 0)
+			(type default)
+		)
+	)
+	(wire
+		(pts
 			(xy 252.73 83.82) (xy 252.73 86.36)
 		)
@@
 	(wire
 		(pts
-			(xy 156.21 49.53) (xy 156.21 48.26)
+			(xy 147.32 49.53) (xy 147.32 48.26)
 		)
 		(stroke
@@
 	(wire
 		(pts
-			(xy 156.21 58.42) (xy 175.26 58.42)
-		)
-		(stroke
-			(width 0)
-			(type default)
-		)
-	)
-	(wire
-		(pts
 			(xy 189.23 60.96) (xy 200.66 60.96)
 		)
@@
 	(wire
 		(pts
-			(xy 146.05 54.61) (xy 146.05 58.42)
+			(xy 137.16 54.61) (xy 137.16 58.42)
 		)
 		(stroke
@@
 	(wire
 		(pts
-			(xy 146.05 49.53) (xy 146.05 48.26)
+			(xy 137.16 49.53) (xy 137.16 48.26)
 		)
 		(stroke
@@
 	(wire
 		(pts
-			(xy 156.21 54.61) (xy 156.21 58.42)
+			(xy 147.32 54.61) (xy 147.32 58.42)
 		)
 		(stroke
@@
 	)
 	(symbol
+		(lib_id "Diode:1N5819WS")
+		(at 156.21 58.42 0)
+		(mirror y)
+		(unit 1)
+		(exclude_from_sim no)
+		(in_bom yes)
+		(on_board yes)
+		(dnp no)
+		(property "Reference" "D1"
+			(at 156.5275 64.77 0)
+			(effects
+				(font
+					(size 1.27 1.27)
+				)
+			)
+		)
+		(property "Value" "B5819"
+			(at 156.5275 62.23 0)
+			(effects
+				(font
+					(size 1.27 1.27)
+				)
+			)
+		)
+		(property "Footprint" "Diode_SMD:D_SOD-323_HandSoldering"
+			(at 156.21 62.865 0)
+			(effects
+				(font
+					(size 1.27 1.27)
+				)
+				(hide yes)
+			)
+		)
+		(property "Datasheet" ""
+			(at 156.21 58.42 0)
+			(effects
+				(font
+					(size 1.27 1.27)
+				)
+				(hide yes)
+			)
+		)
+		(property "Description" ""
+			(at 156.21 58.42 0)
+			(effects
+				(font
+					(size 1.27 1.27)
+				)
+				(hide yes)
+			)
+		)
+		(property "JLCPCB Part #" "C64886"
+			(at 156.21 58.42 0)
+			(effects
+				(font
+					(size 1.27 1.27)
+				)
+				(hide yes)
+			)
+		)
+		(property "MFR. Part #" "B5819WS"
+			(at 156.21 58.42 0)
+			(effects
+				(font
+					(size 1.27 1.27)
+				)
+				(hide yes)
+			)
+		)
+		(pin "1"
+		)
+		(pin "2"
+		)
+		(instances
+			(project ""
+				(path "/53f9535d-094b-439f-baf7-92a0b9b7a939/2e2155ce-e3ba-4327-89a0-259f1fcfea4e"
+					(reference "D1")
+					(unit 1)
+				)
+			)
+		)
+	)
+	(symbol
 		(lib_id "Device:C_Small")
 		(at 200.66 64.77 0)
@@
 	(symbol
 		(lib_id "Device:R_Small")
-		(at 146.05 52.07 0)
+		(at 137.16 52.07 0)
 		(mirror y)
 		(unit 1)
@@
 		(dnp no)
 		(property "Reference" "R14"
-			(at 148.59 50.7999 0)
+			(at 139.7 50.7999 0)
 			(effects
 				(font
@@
 		)
 		(property "Value" "0R"
-			(at 148.59 53.3399 0)
+			(at 139.7 53.3399 0)
 			(effects
 				(font
@@
 		)
 		(property "Footprint" "Resistor_SMD:R_0603_1608Metric"
-			(at 146.05 52.07 0)
+			(at 137.16 52.07 0)
 			(effects
 				(font
@@
 		)
 		(property "Datasheet" "~"
-			(at 146.05 52.07 0)
+			(at 137.16 52.07 0)
 			(effects
 				(font
@@
 		)
 		(property "Description" "Resistor, small symbol"
-			(at 146.05 52.07 0)
+			(at 137.16 52.07 0)
 			(effects
 				(font
@@
 		)
 		(property "JLCPCB Part #" "C21189"
-			(at 146.05 52.07 0)
+			(at 137.16 52.07 0)
 			(effects
 				(font
@@
 		)
 		(property "MFR. Part #" "0603WAF0000T5E"
-			(at 146.05 52.07 0)
+			(at 137.16 52.07 0)
 			(effects
 				(font
@@
 		)
 		(property "Cal" ""
-			(at 146.05 52.07 0)
+			(at 137.16 52.07 0)
 			(effects
 				(font
@@
 		)
 		(property "Sim.Pin" ""
-			(at 146.05 52.07 0)
+			(at 137.16 52.07 0)
 			(effects
 				(font
@@
 	(symbol
 		(lib_id "power:+BATT")
-		(at 146.05 48.26 0)
+		(at 137.16 48.26 0)
 		(unit 1)
 		(exclude_from_sim no)
@@
 		(fields_autoplaced yes)
 		(property "Reference" "#PWR036"
-			(at 146.05 52.07 0)
+			(at 137.16 52.07 0)
 			(effects
 				(font
@@
 		)
 		(property "Value" "+BATT"
-			(at 146.05 43.18 0)
+			(at 137.16 43.18 0)
 			(effects
 				(font
@@
 		)
 		(property "Footprint" ""
-			(at 146.05 48.26 0)
+			(at 137.16 48.26 0)
 			(effects
 				(font
@@
 		)
 		(property "Datasheet" ""
-			(at 146.05 48.26 0)
+			(at 137.16 48.26 0)
 			(effects
 				(font
@@
 		)
 		(property "Description" "Power symbol creates a global label with name \"+BATT\""
-			(at 146.05 48.26 0)
+			(at 137.16 48.26 0)
 			(effects
 				(font
@@
 	(symbol
 		(lib_id "Device:R_Small")
-		(at 156.21 52.07 0)
+		(at 147.32 52.07 0)
 		(mirror y)
 		(unit 1)
@@
 		(dnp yes)
 		(property "Reference" "R15"
-			(at 158.75 50.7999 0)
+			(at 149.86 50.7999 0)
 			(effects
 				(font
@@
 		)
 		(property "Value" "0R"
-			(at 158.75 53.3399 0)
+			(at 149.86 53.3399 0)
 			(effects
 				(font
@@
 		)
 		(property "Footprint" "Resistor_SMD:R_0603_1608Metric"
-			(at 156.21 52.07 0)
+			(at 147.32 52.07 0)
 			(effects
 				(font
@@
 		)
 		(property "Datasheet" "~"
-			(at 156.21 52.07 0)
+			(at 147.32 52.07 0)
 			(effects
 				(font
@@
 		)
 		(property "Description" "Resistor, small symbol"
-			(at 156.21 52.07 0)
+			(at 147.32 52.07 0)
 			(effects
 				(font
@@
 		)
 		(property "JLCPCB Part #" "C21189"
-			(at 156.21 52.07 0)
+			(at 147.32 52.07 0)
 			(effects
 				(font
@@
 		)
 		(property "MFR. Part #" "0603WAF0000T5E"
-			(at 156.21 52.07 0)
+			(at 147.32 52.07 0)
 			(effects
 				(font
@@
 		)
 		(property "Cal" ""
-			(at 156.21 52.07 0)
+			(at 147.32 52.07 0)
 			(effects
 				(font
@@
 		)
 		(property "Sim.Pin" ""
-			(at 156.21 52.07 0)
+			(at 147.32 52.07 0)
 			(effects
 				(font
@@
 	(symbol
 		(lib_id "power:VDD")
-		(at 156.21 48.26 0)
+		(at 147.32 48.26 0)
 		(unit 1)
 		(exclude_from_sim no)
@@
 		(fields_autoplaced yes)
 		(property "Reference" "#PWR037"
-			(at 156.21 52.07 0)
+			(at 147.32 52.07 0)
 			(effects
 				(font
@@
 		)
 		(property "Value" "VDDH"
-			(at 156.21 43.18 0)
+			(at 147.32 43.18 0)
 			(effects
 				(font
@@
 		)
 		(property "Footprint" ""
-			(at 156.21 48.26 0)
+			(at 147.32 48.26 0)
 			(effects
 				(font
@@
 		)
 		(property "Datasheet" ""
-			(at 156.21 48.26 0)
+			(at 147.32 48.26 0)
 			(effects
 				(font
@@
 		)
 		(property "Description" "Power symbol creates a global label with name \"VDD\""
-			(at 156.21 48.26 0)
+			(at 147.32 48.26 0)
 			(effects
 				(font

Commit message: feat: add 3D models (USB-C, TRRS, Switch)
Parts:
- SW1: now fitted
- SW2: now not fitted
Changed lines of the file:
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@@
 		(in_bom yes)
 		(on_board yes)
-		(dnp no)
+		(dnp yes)
 		(fields_autoplaced yes)
 		(property "Reference" "SW2"
@@
 		(in_bom yes)
 		(on_board yes)
-		(dnp yes)
+		(dnp no)
 		(fields_autoplaced yes)
 		(property "Reference" "SW1"
