File: rev41/pcb/main_board/main_board.kicad_pcb (KiCad board)
At the start: 2 copper layers, 86 parts, among them J1 Conn_02x10_Odd_Even, J2 Conn_02x10_Odd_Even, J3 Conn_01x08, SW1 SW_Push_45deg, SW10 SW_Push_45deg, SW11 SW_Push_45deg, SW12 SW_Push_45deg, SW13 SW_Push_45deg, SW14 SW_Push_45deg, SW15 SW_Push_45deg, SW16 SW_Push_45deg, SW17 SW_Push_45deg, SW18 SW_Push_45deg, SW19 SW_Push_45deg, SW2 SW_Push_45deg, SW20 SW_Push_45deg, SW21 SW_Push_45deg, SW22 SW_Push_45deg, SW23 SW_Push_45deg, SW24 SW_Push_45deg, SW25 SW_Push_45deg, SW26 SW_Push_45deg, SW27 SW_Push_45deg, SW28 SW_Push_45deg, SW29 SW_Push_45deg, SW3 SW_Push_45deg, SW4 SW_Push_45deg, SW5 SW_Push_45deg, SW6 SW_Push_45deg, SW7 SW_Push_45deg, SW8 SW_Push_45deg, SW9 SW_Push_45deg

Commit message: feat: update placement
Parts:
- removed J3: Conn_01x08, ErgoSNM_Keyboard:FPC_8P_0.5mm_AFC01-S08FCA-00
- H1, H2, H3, H4, H5, H6: moved to F.Cu
- moved H4 269.9 mm to (187.3, 120.0), turned to 0 degrees
- moved H3 264.0 mm to (187.3, 62.9), turned to 0 degrees
- moved H5 254.5 mm to (168.9, 100.8), turned to 0 degrees
- moved H6 213.1 mm to (130.8, 74.7), turned to 0 degrees
- moved H2 190.2 mm to (111.8, 115.3), turned to 0 degrees
- moved TP7 172.4 mm to (128.0, 132.1)
- moved TP10 172.3 mm to (187.2, 135.9)
- moved TP11 172.2 mm to (205.5, 136.1)
- moved TP8 170.2 mm to (149.4, 128.8)
- moved TP9 169.1 mm to (168.1, 131.1)
- moved TP6 159.0 mm to (108.5, 115.6)
- moved TP1 112.8 mm to (205.5, 46.0)
- moved TP2 111.7 mm to (205.5, 65.0)
- moved TP3 111.7 mm to (205.5, 84.1)
- moved TP4 111.7 mm to (205.5, 103.1)
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- renumbered TP9 to TP10, TP10 to TP11, TP11 to TP9
Other:
- board outline added: 116.1 x 100.8 mm
