File: rev41/pcb/main_board/main_board.kicad_sch (KiCad schematic)
At the start: 0 parts

Commit message: feat: add basic parts
Parts:
- added BTN1, BTN2: RESET, Button_Switch_SMD:SW_SPST_TL3342, symbol Switch:SW_Push
- added D1, D10, D11, D12, D13, D14, D15, D16, D17, D18, D19, D2, D20, D21, D22, D23, D24, D25, D26, D27, D28, D29, D3, D4, D5, D6, D7, D8, D9: 1N4148WS, Diode_SMD:D_SOD-323_HandSoldering, symbol Diode:1N4148W
- added H1, H2, H3, H4, H5, H6: MountingHole, MountingHole:MountingHole_2.2mm_M2_ISO14580, symbol Mechanical:MountingHole
- added J1, J2: Conn_02x10_Odd_Even, Connector_PinSocket_1.27mm:PinSocket_2x10_P1.27mm_Vertical, symbol Connector_Generic:Conn_02x10_Odd_Even
- added J3: Conn_01x08, ErgoSNM_Keyboard:FPC_8P_0.5mm_AFC01-S08FCA-00, symbol Connector_Generic:Conn_01x08
- added LD1, LD2, LD3, LD4: LED, LED_SMD:LED_0603_1608Metric, symbol Device:LED
- added R1, R2: 10k, Resistor_SMD:R_0402_1005Metric, symbol Device:R
- added SW1, SW10, SW11, SW12, SW13, SW14, SW15, SW16, SW17, SW18, SW19, SW2, SW20, SW21, SW22, SW23, SW24, SW25, SW26, SW27, SW28, SW29, SW3, SW4, SW5, SW6, SW7, SW8, SW9: SW_Push_45deg, key-switches:SW_MX_Kailh_Choc_V1V2_HotSwap_Hybrid_double, symbol Switch:SW_Push_45deg
- added TP1: R0, TestPoint:TestPoint_Pad_D1.0mm, symbol Connector:TestPoint
- added TP10: C5, TestPoint:TestPoint_Pad_D1.0mm, symbol Connector:TestPoint
- added TP11: C3, TestPoint:TestPoint_Pad_D1.0mm, symbol Connector:TestPoint
- added TP2: R1, TestPoint:TestPoint_Pad_D1.0mm, symbol Connector:TestPoint
- added TP3: R2, TestPoint:TestPoint_Pad_D1.0mm, symbol Connector:TestPoint
- added TP4: R3, TestPoint:TestPoint_Pad_D1.0mm, symbol Connector:TestPoint
- added TP5: R4, TestPoint:TestPoint_Pad_D1.0mm, symbol Connector:TestPoint
- added TP6: C0, TestPoint:TestPoint_Pad_D1.0mm, symbol Connector:TestPoint
- added TP7: C1, TestPoint:TestPoint_Pad_D1.0mm, symbol Connector:TestPoint
- added TP8: C2, TestPoint:TestPoint_Pad_D1.0mm, symbol Connector:TestPoint
- added TP9: C4, TestPoint:TestPoint_Pad_D1.0mm, symbol Connector:TestPoint
Connections:
- new net: D3.2 (A), SW3.2
- new net: D7.2 (A), SW7.2
- new net: D17.2 (A), SW17.2
- new net: D4.2 (A), SW4.2
- new net: D25.2 (A), SW25.2
- new net: D14.2 (A), SW14.2
- new net: D19.2 (A), SW19.2
- new net: LD1.1 (K), LD2.1 (K), R1.1
- new net: D16.2 (A), SW16.2
- new net: D26.2 (A), SW26.2
- new net: D22.2 (A), SW22.2
- new net: D5.2 (A), SW5.2
- new net: D28.2 (A), SW28.2
- new net: D10.2 (A), SW10.2
- new net: D11.2 (A), SW11.2
- new net: D23.2 (A), SW23.2
- new net: D29.2 (A), SW29.2
- new net: D8.2 (A), SW8.2
- new net: D27.2 (A), SW27.2
- new net: D6.2 (A), SW6.2
- new net: D1.2 (A), SW1.2
- new net: D24.2 (A), SW24.2
- new net: LD3.1 (K), LD4.1 (K), R2.1
- new net: D18.2 (A), SW18.2
- new net: D21.2 (A), SW21.2
- new net: D15.2 (A), SW15.2
- new net: D20.2 (A), SW20.2
- new net: D13.2 (A), SW13.2
- new net: D12.2 (A), SW12.2
- new net: D9.2 (A), SW9.2
- new net: D2.2 (A), SW2.2
- new net COL_0: J1.8 (Pin_8), SW1.1, SW13.1, SW19.1, SW7.1, TP6.1
- new net COL_1: J1.6 (Pin_6), SW14.1, SW2.1, SW20.1, SW25.1, SW8.1, TP7.1
- new net COL_2: J1.10 (Pin_10), SW15.1, SW21.1, SW26.1, SW3.1, SW9.1, TP8.1
- new net COL_3: J1.16 (Pin_16), SW10.1, SW16.1, SW22.1, SW27.1, SW4.1, TP11.1
- new net COL_4: J1.14 (Pin_14), SW11.1, SW17.1, SW23.1, SW28.1, SW5.1, TP9.1
- new net COL_5: J1.12 (Pin_12), SW12.1, SW18.1, SW24.1, SW29.1, SW6.1, TP10.1
- new net GND: BTN1.1, BTN2.1, J2.2 (Pin_2), J2.20 (Pin_20), R1.2, R2.2
- new net LED_1: J1.18 (Pin_18), LD1.2 (A), LD2.2 (A)
- new net LED_2: J1.20 (Pin_20), LD3.2 (A), LD4.2 (A)
- new net RESET: BTN1.2, BTN2.2, J2.17 (Pin_17), J2.3 (Pin_3)
- new net ROW_0: D1.1 (K), D2.1 (K), D3.1 (K), D4.1 (K), D5.1 (K), D6.1 (K), J1.5 (Pin_5), TP1.1
- new net ROW_1: D10.1 (K), D11.1 (K), D12.1 (K), D7.1 (K), D8.1 (K), D9.1 (K), J1.7 (Pin_7), TP2.1
- new net ROW_2: D13.1 (K), D14.1 (K), D15.1 (K), D16.1 (K), D17.1 (K), D18.1 (K), J1.9 (Pin_9), TP3.1
- new net ROW_3: D19.1 (K), D20.1 (K), D21.1 (K), D22.1 (K), D23.1 (K), D24.1 (K), J1.11 (Pin_11), TP4.1
- new net ROW_4: D25.1 (K), D26.1 (K), D27.1 (K), D28.1 (K), D29.1 (K), J1.13 (Pin_13), TP5.1
- new net ROW_5: J1.15 (Pin_15)
- new net VDD: J2.1 (Pin_1), J2.19 (Pin_19)
Other:
- company: (none) -> SideraKB
- title: (none) -> ErgoSNM Keyboard - Main Board

Commit message: feat: update placement
Parts:
- removed J3: Conn_01x08, ErgoSNM_Keyboard:FPC_8P_0.5mm_AFC01-S08FCA-00, symbol Connector_Generic:Conn_01x08
- renumbered TP9 to TP10, TP10 to TP11, TP11 to TP9
Other:
- moved on the sheet: TP10, TP11, TP7, TP8, TP9
Changed lines of the file:
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@@
 	(wire
 		(pts
-			(xy 88.9 139.7) (xy 88.9 154.94)
+			(xy 88.9 139.7) (xy 88.9 156.21)
 		)
 		(stroke
@@
 	(wire
 		(pts
-			(xy 165.1 139.7) (xy 165.1 154.94)
+			(xy 165.1 139.7) (xy 165.1 156.21)
 		)
 		(stroke
@@
 	(wire
 		(pts
-			(xy 114.3 139.7) (xy 114.3 155.0214)
+			(xy 114.3 139.7) (xy 114.3 156.21)
 		)
 		(stroke
@@
 	(wire
 		(pts
-			(xy 139.7 139.7) (xy 139.7 154.94)
+			(xy 139.7 139.7) (xy 139.7 156.21)
 		)
 		(stroke
@@
 	(wire
 		(pts
-			(xy 63.5 139.7) (xy 63.5 154.94)
+			(xy 63.5 139.7) (xy 63.5 156.21)
 		)
 		(stroke
@@
 		)
 		(instances
-			(project ""
+			(project "main_board"
 				(path "/2a2761ca-cea7-46c5-81c5-d1241812e760"
 					(reference "TP6")
@@
 		)
 		(instances
-			(project ""
+			(project "main_board"
 				(path "/2a2761ca-cea7-46c5-81c5-d1241812e760"
 					(reference "R1")
@@
 	(symbol
 		(lib_id "Connector:TestPoint")
-		(at 139.7 154.94 180)
+		(at 139.7 156.21 180)
 		(unit 1)
 		(exclude_from_sim no)
@@
 		(dnp no)
 		(fields_autoplaced yes)
-		(property "Reference" "TP9"
-			(at 142.24 156.9719 0)
+		(property "Reference" "TP10"
+			(at 142.24 158.2419 0)
 			(effects
 				(font
@@
 		)
 		(property "Value" "C4"
-			(at 142.24 159.5119 0)
+			(at 142.24 160.7819 0)
 			(effects
 				(font
@@
 		)
 		(property "Footprint" "TestPoint:TestPoint_Pad_D1.0mm"
-			(at 134.62 154.94 0)
+			(at 134.62 156.21 0)
 			(effects
 				(font
@@
 		)
 		(property "Datasheet" "~"
-			(at 134.62 154.94 0)
+			(at 134.62 156.21 0)
 			(effects
 				(font
@@
 		)
 		(property "Description" "test point"
-			(at 139.7 154.94 0)
+			(at 139.7 156.21 0)
 			(effects
 				(font
@@
 			(project "main_board"
 				(path "/2a2761ca-cea7-46c5-81c5-d1241812e760"
-					(reference "TP9")
+					(reference "TP10")
 					(unit 1)
 				)
@@
 	)
 	(symbol
-		(lib_id "Connector_Generic:Conn_01x08")
-		(at 237.49 128.27 0)
-		(unit 1)
-		(exclude_from_sim no)
-		(in_bom yes)
-		(on_board yes)
-		(dnp no)
-		(fields_autoplaced yes)
-		(property "Reference" "J3"
-			(at 240.03 128.2699 0)
-			(effects
-				(font
-					(size 1.27 1.27)
-				)
-				(justify left)
-			)
-		)
-		(property "Value" "Conn_01x08"
-			(at 240.03 130.8099 0)
-			(effects
-				(font
-					(size 1.27 1.27)
-				)
-				(justify left)
-			)
-		)
-		(property "Footprint" "ErgoSNM_Keyboard:FPC_8P_0.5mm_AFC01-S08FCA-00"
-			(at 237.49 128.27 0)
-			(effects
-				(font
-					(size 1.27 1.27)
-				)
-				(hide yes)
-			)
-		)
-		(property "Datasheet" "~"
-			(at 237.49 128.27 0)
-			(effects
-				(font
-					(size 1.27 1.27)
-				)
-				(hide yes)
-			)
-		)
-		(property "Description" "Generic connector, single row, 01x08, script generated (kicad-library-utils/schlib/autogen/connector/)"
-			(at 237.49 128.27 0)
-			(effects
-				(font
-					(size 1.27 1.27)
-				)
-				(hide yes)
-			)
-		)
-		(pin "1"
-		)
-		(pin "5"
-		)
-		(pin "7"
-		)
-		(pin "4"
-		)
-		(pin "8"
-		)
-		(pin "3"
-		)
-		(pin "2"
-		)
-		(pin "6"
-		)
-		(instances
-			(project ""
-				(path "/2a2761ca-cea7-46c5-81c5-d1241812e760"
-					(reference "J3")
-					(unit 1)
-				)
-			)
-		)
-	)
-	(symbol
 		(lib_id "Diode:1N4148W")
 		(at 152.4 46.99 270)
@@
 		)
 		(instances
-			(project ""
+			(project "main_board"
 				(path "/2a2761ca-cea7-46c5-81c5-d1241812e760"
 					(reference "D1")
@@
 		)
 		(instances
-			(project ""
+			(project "main_board"
 				(path "/2a2761ca-cea7-46c5-81c5-d1241812e760"
 					(reference "LD2")
@@
 		)
 		(instances
-			(project ""
+			(project "main_board"
 				(path "/2a2761ca-cea7-46c5-81c5-d1241812e760"
 					(reference "BTN1")
@@
 		)
 		(instances
-			(project ""
+			(project "main_board"
 				(path "/2a2761ca-cea7-46c5-81c5-d1241812e760"
 					(reference "#PWR04")
@@
 		)
 		(instances
-			(project ""
+			(project "main_board"
 				(path "/2a2761ca-cea7-46c5-81c5-d1241812e760"
 					(reference "J1")
@@
 		)
 		(instances
-			(project ""
+			(project "main_board"
 				(path "/2a2761ca-cea7-46c5-81c5-d1241812e760"
 					(reference "H2")
@@
 	(symbol
 		(lib_id "Connector:TestPoint")
-		(at 114.3 155.0214 180)
+		(at 114.3 156.21 180)
 		(unit 1)
 		(exclude_from_sim no)
@@
 		(dnp no)
 		(fields_autoplaced yes)
-		(property "Reference" "TP11"
-			(at 116.84 157.0533 0)
+		(property "Reference" "TP9"
+			(at 116.84 158.2419 0)
 			(effects
 				(font
@@
 		)
 		(property "Value" "C3"
-			(at 116.84 159.5933 0)
+			(at 116.84 160.7819 0)
 			(effects
 				(font
@@
 		)
 		(property "Footprint" "TestPoint:TestPoint_Pad_D1.0mm"
-			(at 109.22 155.0214 0)
+			(at 109.22 156.21 0)
 			(effects
 				(font
@@
 		)
 		(property "Datasheet" "~"
-			(at 109.22 155.0214 0)
+			(at 109.22 156.21 0)
 			(effects
 				(font
@@
 		)
 		(property "Description" "test point"
-			(at 114.3 155.0214 0)
+			(at 114.3 156.21 0)
 			(effects
 				(font
@@
 			(project "main_board"
 				(path "/2a2761ca-cea7-46c5-81c5-d1241812e760"
-					(reference "TP11")
+					(reference "TP9")
 					(unit 1)
 				)
@@
 	(symbol
 		(lib_id "Connector:TestPoint")
-		(at 88.9 154.94 180)
+		(at 88.9 156.21 180)
 		(unit 1)
 		(exclude_from_sim no)
@@
 		(fields_autoplaced yes)
 		(property "Reference" "TP8"
-			(at 91.44 156.9719 0)
+			(at 91.44 158.2419 0)
 			(effects
 				(font
@@
 		)
 		(property "Value" "C2"
-			(at 91.44 159.5119 0)
+			(at 91.44 160.7819 0)
 			(effects
 				(font
@@
 		)
 		(property "Footprint" "TestPoint:TestPoint_Pad_D1.0mm"
-			(at 83.82 154.94 0)
+			(at 83.82 156.21 0)
 			(effects
 				(font
@@
 		)
 		(property "Datasheet" "~"
-			(at 83.82 154.94 0)
+			(at 83.82 156.21 0)
 			(effects
 				(font
@@
 		)
 		(property "Description" "test point"
-			(at 88.9 154.94 0)
+			(at 88.9 156.21 0)
 			(effects
 				(font
@@
 		)
 		(instances
-			(project ""
+			(project "main_board"
 				(path "/2a2761ca-cea7-46c5-81c5-d1241812e760"
 					(reference "SW1")
@@
 	(symbol
 		(lib_id "Connector:TestPoint")
-		(at 165.1 154.94 180)
+		(at 165.1 156.21 180)
 		(unit 1)
 		(exclude_from_sim no)
@@
 		(dnp no)
 		(fields_autoplaced yes)
-		(property "Reference" "TP10"
-			(at 167.64 156.9719 0)
+		(property "Reference" "TP11"
+			(at 167.64 158.2419 0)
 			(effects
 				(font
@@
 		)
 		(property "Value" "C5"
-			(at 167.64 159.5119 0)
+			(at 167.64 160.7819 0)
 			(effects
 				(font
@@
 		)
 		(property "Footprint" "TestPoint:TestPoint_Pad_D1.0mm"
-			(at 160.02 154.94 0)
+			(at 160.02 156.21 0)
 			(effects
 				(font
@@
 		)
 		(property "Datasheet" "~"
-			(at 160.02 154.94 0)
+			(at 160.02 156.21 0)
 			(effects
 				(font
@@
 		)
 		(property "Description" "test point"
-			(at 165.1 154.94 0)
+			(at 165.1 156.21 0)
 			(effects
 				(font
@@
 			(project "main_board"
 				(path "/2a2761ca-cea7-46c5-81c5-d1241812e760"
-					(reference "TP10")
+					(reference "TP11")
 					(unit 1)
 				)
@@
 		)
 		(instances
-			(project ""
+			(project "main_board"
 				(path "/2a2761ca-cea7-46c5-81c5-d1241812e760"
 					(reference "#PWR01")
@@
 	(symbol
 		(lib_id "Connector:TestPoint")
-		(at 63.5 154.94 180)
+		(at 63.5 156.21 180)
 		(unit 1)
 		(exclude_from_sim no)
@@
 		(fields_autoplaced yes)
 		(property "Reference" "TP7"
-			(at 66.04 156.9719 0)
+			(at 66.04 158.2419 0)
 			(effects
 				(font
@@
 		)
 		(property "Value" "C1"
-			(at 66.04 159.5119 0)
+			(at 66.04 160.7819 0)
 			(effects
 				(font
@@
 		)
 		(property "Footprint" "TestPoint:TestPoint_Pad_D1.0mm"
-			(at 58.42 154.94 0)
+			(at 58.42 156.21 0)
 			(effects
 				(font
@@
 		)
 		(property "Datasheet" "~"
-			(at 58.42 154.94 0)
+			(at 58.42 156.21 0)
 			(effects
 				(font
@@
 		)
 		(property "Description" "test point"
-			(at 63.5 154.94 0)
+			(at 63.5 156.21 0)
 			(effects
 				(font
