File: rev41/pcb/main_board/main_board.kicad_sch (KiCad schematic)
At the start: 85 parts, among them J1 Conn_02x10_Odd_Even, J2 Conn_02x10_Odd_Even, SW1 SW_Push_45deg, SW10 SW_Push_45deg, SW11 SW_Push_45deg, SW12 SW_Push_45deg, SW13 SW_Push_45deg, SW14 SW_Push_45deg, SW15 SW_Push_45deg, SW16 SW_Push_45deg, SW17 SW_Push_45deg, SW18 SW_Push_45deg, SW19 SW_Push_45deg, SW2 SW_Push_45deg, SW20 SW_Push_45deg, SW21 SW_Push_45deg, SW22 SW_Push_45deg, SW23 SW_Push_45deg, SW24 SW_Push_45deg, SW25 SW_Push_45deg, SW26 SW_Push_45deg, SW27 SW_Push_45deg, SW28 SW_Push_45deg, SW29 SW_Push_45deg, SW3 SW_Push_45deg, SW4 SW_Push_45deg, SW5 SW_Push_45deg, SW6 SW_Push_45deg, SW7 SW_Push_45deg, SW8 SW_Push_45deg, SW9 SW_Push_45deg

Commit message: feat: basic routed
Connections:
- net COL_0: now also J1.6 (Pin_6); no longer J1.8 (Pin_8)
- net COL_1: now also J1.8 (Pin_8); no longer J1.6 (Pin_6)
- net COL_3: now also J1.12 (Pin_12); no longer J1.16 (Pin_16)
- net COL_5: now also J1.16 (Pin_16); no longer J1.12 (Pin_12)
- no-connect marks 0 -> 20

Commit message: feat: update BOM
Parts:
- BTN1, BTN2: JLCPCB Part # (none) -> C318884; MFR. Part # (none) -> TS-1187A-B-A-B
- D1, D10, D11, D12, D13, D14, D15, D16, D17, D18, D19, D2, D20, D21, D22, D23, D24, D25, D26, D27, D28, D29, D3, D4, D5, D6, D7, D8, D9: JLCPCB Part # (none) -> C2128; MFR. Part # (none) -> 1N4148WS
- J1, J2, TP1, TP10, TP11, TP2, TP3, TP4, TP5, TP6, TP7, TP8, TP9: now left out of the parts list
- R1, R2: JLCPCB Part # (none) -> C25744; MFR. Part # (none) -> 0402WGF1002TCE
