File: rev41/pcb/core_board_e73/power.kicad_sch (KiCad schematic)
At the start: 36 parts, among them J8 Conn_Batt, J9 USB_C_Receptacle_USB2.0_16P, SW1 SW_SPDT, SW2 SW_SPDT, U2 BQ24075RGT, U3 TPS63900, U4 USBLC6-2SC6

Commit message: feat: core board e73 basic routed
Parts:
- U3: footprint Package_SON:WSON-10-1EP_2.5x2.5mm_P0.5mm_EP1.2x2mm_ThermalVias -> Package_SON:WSON-10-1EP_2.5x2.5mm_P0.5mm_EP1.2x2mm
Changed lines of the file:
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@@
 			)
 		)
-		(property "Footprint" "Package_SON:WSON-10-1EP_2.5x2.5mm_P0.5mm_EP1.2x2mm_ThermalVias"
+		(property "Footprint" "Package_SON:WSON-10-1EP_2.5x2.5mm_P0.5mm_EP1.2x2mm"
 			(at 231.14 77.47 0)
 			(hide yes)

Commit message: feat: update BOM
Parts:
- C10, C8: JLCPCB Part # (none) -> C45783; MFR. Part # (none) -> CL21A226MAQNNNE
- C11: JLCPCB Part # (none) -> C1525; MFR. Part # (none) -> CL05B104KO5NNNC
- C12: JLCPCB Part # (none) -> C1744; MFR. Part # (none) -> 0805B472K500NT
- C6: JLCPCB Part # (none) -> C52923; MFR. Part # (none) -> CL05A105KA5NQNC
- C7, C9: JLCPCB Part # (none) -> C23733; MFR. Part # (none) -> CL05A475MP5NRNC
- D1: JLCPCB Part # (none) -> C64886; MFR. Part # (none) -> B5819WS
- F1: JLCPCB Part # (none) -> C269104; MFR. Part # (none) -> SMD0805B050TF
- J8: JLCPCB Part # (none) -> C295747; MFR. Part # (none) -> S2B-PH-SM4-TB(LF)(SN)
- J9: JLCPCB Part # (none) -> C165948; MFR. Part # (none) -> TYPE-C-31-M-12
- L1: JLCPCB Part # (none) -> C5179446; MFR. Part # (none) -> FWP252012P-2R2ML
- R10, R12, R9: JLCPCB Part # (none) -> C25744; MFR. Part # (none) -> 0402WGF1002TCE
- R11: JLCPCB Part # (none) -> C4109; MFR. Part # (none) -> 0402WGF2001TCE
- R13: JLCPCB Part # (none) -> C22809; MFR. Part # (none) -> 0603WAF1502T5E
- R14, R4, R5, R6, R7, R8: JLCPCB Part # (none) -> C21189; MFR. Part # (none) -> 0603WAF0000T5E
- R15: JLCPCB Part # (none) -> C4184; MFR. Part # (none) -> 0603WAF2002T5E
- R16, R17: JLCPCB Part # (none) -> C25905; MFR. Part # (none) -> 0402WGF5101TCE
- R18: JLCPCB Part # (none) -> C22935; MFR. Part # (none) -> 0603WAF1004T5E
- U2: JLCPCB Part # (none) -> C15464; MFR. Part # (none) -> BQ24075RGTR
- U3: JLCPCB Part # (none) -> C1518762; MFR. Part # (none) -> TPS63900DSKR
- U4: JLCPCB Part # (none) -> C2687116; MFR. Part # (none) -> USBLC6-2SC6; Rotation Offset (none) -> 90
