File: rev41/pcb/thumb_cluster/thumb_cluster.kicad_sch (KiCad schematic)
At the start: 23 parts, among them J1 Conn, J2 Conn, SW1 SW_Push_45deg, SW2 SW_Push_45deg, SW3 SW_Push_45deg, SW4 SW_Push_45deg, SW5 SW_Push_45deg, SW6 SW_Push_45deg, SW7 SW_Push_45deg, SW8 SW_Push_45deg

Commit message: feat: update title block
Other:
- company: (none) -> SideraKB
- title: (none) -> ErgoSNM Keyboard - Thumb Cluster
Changed lines of the file:
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@@
 	(generator_version "10.0")
 	(paper "A4")
+	(title_block
+		(title "ErgoSNM Keyboard - Thumb Cluster")
+		(rev "4.1.A")
+		(company "SideraKB")
+		(comment 1 "Open source hardware, CERN-OHL-P_v2")
+		(comment 2 "https://github.com/siderakb/ergo-snm-keyboard")
+	)
 	(junction
 		(at 184.15 63.5)

Commit message: feat: update BOM
Parts:
- D1, D2, D3, D4, D5, D6, D7, D8: JLCPCB Part # (none) -> C2128; MFR. Part # (none) -> 1N4148WS
- J1, J2: JLCPCB Part # (none) -> C2856797; MFR. Part # (none) -> FPC-05F-8PH20
